File: V1/esp-poe-010v-V1-power.kicad_sch (KiCad schematic)
At the start: 32 parts, among them U1 TPS2376DDAR-H, U2 TX4138, U3 SY8089A1AAC

Commit message: dev time
Other:
- title: ESP 2x Relay Output Module with PoE -> ESP 2x 0-10V Output Module with PoE
Changed lines of the file:
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@@
 	(paper "A4")
 	(title_block
-		(title "ESP 2x Relay Output Module with PoE")
-		(date "2025-06-29")
-		(rev "V1.3")
+		(title "ESP 2x 0-10V Output Module with PoE")
+		(date "2025-12-13")
+		(rev "V1.0")
 	)
 	(text "R_{TPS1}"
@@
 		)
 		(instances
-			(project "esp-poe-2rl-V1"
+			(project "esp-poe-010v-V1"
 				(path "/2bc5a21a-1d79-419d-a592-6852cc07b00a/2ac7b96d-5459-407c-a3e3-5692241632df"
 					(reference "#PWR0156")
@@
 		)
 		(instances
-			(project "esp-poe-2rl-V1"
+			(project "esp-poe-010v-V1"
 				(path "/2bc5a21a-1d79-419d-a592-6852cc07b00a/2ac7b96d-5459-407c-a3e3-5692241632df"
 					(reference "C8")
@@
 		)
 		(instances
-			(project "esp-poe-2rl-V1"
+			(project "esp-poe-010v-V1"
 				(path "/2bc5a21a-1d79-419d-a592-6852cc07b00a/2ac7b96d-5459-407c-a3e3-5692241632df"
 					(reference "R8")
@@
 		)
 		(instances
-			(project "esp-poe-2rl-V1"
+			(project "esp-poe-010v-V1"
 				(path "/2bc5a21a-1d79-419d-a592-6852cc07b00a/2ac7b96d-5459-407c-a3e3-5692241632df"
 					(reference "#PWR0162")
@@
 		)
 		(instances
-			(project "esp-poe-2rl-V1"
+			(project "esp-poe-010v-V1"
 				(path "/2bc5a21a-1d79-419d-a592-6852cc07b00a/2ac7b96d-5459-407c-a3e3-5692241632df"
 					(reference "C3")
@@
 		)
 		(instances
-			(project "esp-poe-2rl-V1"
+			(project "esp-poe-010v-V1"
 				(path "/2bc5a21a-1d79-419d-a592-6852cc07b00a/2ac7b96d-5459-407c-a3e3-5692241632df"
 					(reference "R10")
@@
 		)
 		(instances
-			(project "esp-poe-2rl-V1"
+			(project "esp-poe-010v-V1"
 				(path "/2bc5a21a-1d79-419d-a592-6852cc07b00a/2ac7b96d-5459-407c-a3e3-5692241632df"
 					(reference "#PWR0157")
@@
 		)
 		(instances
-			(project "esp-poe-2rl-V1"
+			(project "esp-poe-010v-V1"
 				(path "/2bc5a21a-1d79-419d-a592-6852cc07b00a/2ac7b96d-5459-407c-a3e3-5692241632df"
 					(reference "L2")
@@
 		)
 		(instances
-			(project "esp-poe-2rl-V1"
+			(project "esp-poe-010v-V1"
 				(path "/2bc5a21a-1d79-419d-a592-6852cc07b00a/2ac7b96d-5459-407c-a3e3-5692241632df"
 					(reference "C1")
@@
 		)
 		(instances
-			(project "esp-poe-2rl-V1"
+			(project "esp-poe-010v-V1"
 				(path "/2bc5a21a-1d79-419d-a592-6852cc07b00a/2ac7b96d-5459-407c-a3e3-5692241632df"
 					(reference "C9")
@@
 		)
 		(instances
-			(project "esp-poe-2rl-V1"
+			(project "esp-poe-010v-V1"
 				(path "/2bc5a21a-1d79-419d-a592-6852cc07b00a/2ac7b96d-5459-407c-a3e3-5692241632df"
 					(reference "#PWR0158")
@@
 		)
 		(instances
-			(project "esp-poe-2rl-V1"
+			(project "esp-poe-010v-V1"
 				(path "/2bc5a21a-1d79-419d-a592-6852cc07b00a/2ac7b96d-5459-407c-a3e3-5692241632df"
 					(reference "#PWR0160")
@@
 		)
 		(instances
-			(project "esp-poe-2rl-V1"
+			(project "esp-poe-010v-V1"
 				(path "/2bc5a21a-1d79-419d-a592-6852cc07b00a/2ac7b96d-5459-407c-a3e3-5692241632df"
 					(reference "D3")
@@
 		)
 		(instances
-			(project "esp-poe-2rl-V1"
+			(project "esp-poe-010v-V1"
 				(path "/2bc5a21a-1d79-419d-a592-6852cc07b00a/2ac7b96d-5459-407c-a3e3-5692241632df"
 					(reference "R1")
@@
 		)
 		(instances
-			(project "esp-poe-2rl-V1"
+			(project "esp-poe-010v-V1"
 				(path "/2bc5a21a-1d79-419d-a592-6852cc07b00a/2ac7b96d-5459-407c-a3e3-5692241632df"
 					(reference "L1")
@@
 		)
 		(instances
-			(project "esp-poe-2rl-V1"
+			(project "esp-poe-010v-V1"
 				(path "/2bc5a21a-1d79-419d-a592-6852cc07b00a/2ac7b96d-5459-407c-a3e3-5692241632df"
 					(reference "R6")
@@
 		)
 		(instances
-			(project "esp-poe-2rl-V1"
+			(project "esp-poe-010v-V1"
 				(path "/2bc5a21a-1d79-419d-a592-6852cc07b00a/2ac7b96d-5459-407c-a3e3-5692241632df"
 					(reference "C7")
@@
 		)
 		(instances
-			(project "esp-poe-2rl-V1"
+			(project "esp-poe-010v-V1"
 				(path "/2bc5a21a-1d79-419d-a592-6852cc07b00a/2ac7b96d-5459-407c-a3e3-5692241632df"
 					(reference "U1")
@@
 		)
 		(instances
-			(project "esp-poe-2rl-V1"
+			(project "esp-poe-010v-V1"
 				(path "/2bc5a21a-1d79-419d-a592-6852cc07b00a/2ac7b96d-5459-407c-a3e3-5692241632df"
 					(reference "C2")
@@
 		)
 		(instances
-			(project "esp-poe-2rl-V1"
+			(project "esp-poe-010v-V1"
 				(path "/2bc5a21a-1d79-419d-a592-6852cc07b00a/2ac7b96d-5459-407c-a3e3-5692241632df"
 					(reference "#FLG0105")
@@
 		)
 		(instances
-			(project "esp-poe-2rl-V1"
+			(project "esp-poe-010v-V1"
 				(path "/2bc5a21a-1d79-419d-a592-6852cc07b00a/2ac7b96d-5459-407c-a3e3-5692241632df"
 					(reference "R3")
@@
 		)
 		(instances
-			(project "esp-poe-2rl-V1"
+			(project "esp-poe-010v-V1"
 				(path "/2bc5a21a-1d79-419d-a592-6852cc07b00a/2ac7b96d-5459-407c-a3e3-5692241632df"
 					(reference "#PWR0155")
@@
 		)
 		(instances
-			(project "esp-poe-2rl-V1"
+			(project "esp-poe-010v-V1"
 				(path "/2bc5a21a-1d79-419d-a592-6852cc07b00a/2ac7b96d-5459-407c-a3e3-5692241632df"
 					(reference "D2")
@@
 		)
 		(instances
-			(project "esp-poe-2rl-V1"
+			(project "esp-poe-010v-V1"
 				(path "/2bc5a21a-1d79-419d-a592-6852cc07b00a/2ac7b96d-5459-407c-a3e3-5692241632df"
 					(reference "#PWR0150")
@@
 		)
 		(instances
-			(project "esp-poe-2rl-V1"
+			(project "esp-poe-010v-V1"
 				(path "/2bc5a21a-1d79-419d-a592-6852cc07b00a/2ac7b96d-5459-407c-a3e3-5692241632df"
 					(reference "R5")
@@
 		)
 		(instances
-			(project "esp-poe-2rl-V1"
+			(project "esp-poe-010v-V1"
 				(path "/2bc5a21a-1d79-419d-a592-6852cc07b00a/2ac7b96d-5459-407c-a3e3-5692241632df"
 					(reference "#PWR0164")
@@
 		)
 		(instances
-			(project "esp-poe-2rl-V1"
+			(project "esp-poe-010v-V1"
 				(path "/2bc5a21a-1d79-419d-a592-6852cc07b00a/2ac7b96d-5459-407c-a3e3-5692241632df"
 					(reference "R9")
@@
 		)
 		(instances
-			(project "esp-poe-2rl-V1"
+			(project "esp-poe-010v-V1"
 				(path "/2bc5a21a-1d79-419d-a592-6852cc07b00a/2ac7b96d-5459-407c-a3e3-5692241632df"
 					(reference "R12")
@@
 		)
 		(instances
-			(project "esp-poe-2rl-V1"
+			(project "esp-poe-010v-V1"
 				(path "/2bc5a21a-1d79-419d-a592-6852cc07b00a/2ac7b96d-5459-407c-a3e3-5692241632df"
 					(reference "R4")
@@
 		)
 		(instances
-			(project "esp-poe-2rl-V1"
+			(project "esp-poe-010v-V1"
 				(path "/2bc5a21a-1d79-419d-a592-6852cc07b00a/2ac7b96d-5459-407c-a3e3-5692241632df"
 					(reference "R7")
@@
 		)
 		(instances
-			(project "esp-poe-2rl-V1"
+			(project "esp-poe-010v-V1"
 				(path "/2bc5a21a-1d79-419d-a592-6852cc07b00a/2ac7b96d-5459-407c-a3e3-5692241632df"
 					(reference "R2")
@@
 		)
 		(instances
-			(project "esp-poe-2rl-V1"
+			(project "esp-poe-010v-V1"
 				(path "/2bc5a21a-1d79-419d-a592-6852cc07b00a/2ac7b96d-5459-407c-a3e3-5692241632df"
 					(reference "D1")
@@
 		)
 		(instances
-			(project "esp-poe-2rl-V1"
+			(project "esp-poe-010v-V1"
 				(path "/2bc5a21a-1d79-419d-a592-6852cc07b00a/2ac7b96d-5459-407c-a3e3-5692241632df"
 					(reference "D5")
@@
 		)
 		(instances
-			(project "esp-poe-2rl-V1"
+			(project "esp-poe-010v-V1"
 				(path "/2bc5a21a-1d79-419d-a592-6852cc07b00a/2ac7b96d-5459-407c-a3e3-5692241632df"
 					(reference "R11")
@@
 		)
 		(instances
-			(project "esp-poe-2rl-V1"
+			(project "esp-poe-010v-V1"
 				(path "/2bc5a21a-1d79-419d-a592-6852cc07b00a/2ac7b96d-5459-407c-a3e3-5692241632df"
 					(reference "U2")
@@
 		)
 		(instances
-			(project "esp-poe-2rl-V1"
+			(project "esp-poe-010v-V1"
 				(path "/2bc5a21a-1d79-419d-a592-6852cc07b00a/2ac7b96d-5459-407c-a3e3-5692241632df"
 					(reference "#PWR0153")
@@
 		)
 		(instances
-			(project "esp-poe-2rl-V1"
+			(project "esp-poe-010v-V1"
 				(path "/2bc5a21a-1d79-419d-a592-6852cc07b00a/2ac7b96d-5459-407c-a3e3-5692241632df"
 					(reference "R13")
@@
 		)
 		(instances
-			(project "esp-poe-2rl-V1"
+			(project "esp-poe-010v-V1"
 				(path "/2bc5a21a-1d79-419d-a592-6852cc07b00a/2ac7b96d-5459-407c-a3e3-5692241632df"
 					(reference "#PWR0152")
@@
 		)
 		(instances
-			(project "esp-poe-2rl-V1"
+			(project "esp-poe-010v-V1"
 				(path "/2bc5a21a-1d79-419d-a592-6852cc07b00a/2ac7b96d-5459-407c-a3e3-5692241632df"
 					(reference "#PWR0151")
@@
 		)
 		(instances
-			(project "esp-poe-2rl-V1"
+			(project "esp-poe-010v-V1"
 				(path "/2bc5a21a-1d79-419d-a592-6852cc07b00a/2ac7b96d-5459-407c-a3e3-5692241632df"
 					(reference "C4")
@@
 		)
 		(instances
-			(project "esp-poe-2rl-V1"
+			(project "esp-poe-010v-V1"
 				(path "/2bc5a21a-1d79-419d-a592-6852cc07b00a/2ac7b96d-5459-407c-a3e3-5692241632df"
 					(reference "U3")
@@
 		)
 		(instances
-			(project "esp-poe-2rl-V1"
+			(project "esp-poe-010v-V1"
 				(path "/2bc5a21a-1d79-419d-a592-6852cc07b00a/2ac7b96d-5459-407c-a3e3-5692241632df"
 					(reference "#PWR0154")
@@
 		)
 		(instances
-			(project "esp-poe-2rl-V1"
+			(project "esp-poe-010v-V1"
 				(path "/2bc5a21a-1d79-419d-a592-6852cc07b00a/2ac7b96d-5459-407c-a3e3-5692241632df"
 					(reference "C5")
@@
 		)
 		(instances
-			(project "esp-poe-2rl-V1"
+			(project "esp-poe-010v-V1"
 				(path "/2bc5a21a-1d79-419d-a592-6852cc07b00a/2ac7b96d-5459-407c-a3e3-5692241632df"
 					(reference "D4")
@@
 		)
 		(instances
-			(project "esp-poe-2rl-V1"
+			(project "esp-poe-010v-V1"
 				(path "/2bc5a21a-1d79-419d-a592-6852cc07b00a/2ac7b96d-5459-407c-a3e3-5692241632df"
 					(reference "#PWR0163")
@@
 		)
 		(instances
-			(project "esp-poe-2rl-V1"
+			(project "esp-poe-010v-V1"
 				(path "/2bc5a21a-1d79-419d-a592-6852cc07b00a/2ac7b96d-5459-407c-a3e3-5692241632df"
 					(reference "C6")
@@
 		)
 		(instances
-			(project "esp-poe-2rl-V1"
+			(project "esp-poe-010v-V1"
 				(path "/2bc5a21a-1d79-419d-a592-6852cc07b00a/2ac7b96d-5459-407c-a3e3-5692241632df"
 					(reference "#PWR0159")
@@
 		)
 		(instances
-			(project "esp-poe-2rl-V1"
+			(project "esp-poe-010v-V1"
 				(path "/2bc5a21a-1d79-419d-a592-6852cc07b00a/2ac7b96d-5459-407c-a3e3-5692241632df"
 					(reference "#FLG0104")
@@
 		)
 		(instances
-			(project "esp-poe-2rl-V1"
+			(project "esp-poe-010v-V1"
 				(path "/2bc5a21a-1d79-419d-a592-6852cc07b00a/2ac7b96d-5459-407c-a3e3-5692241632df"
 					(reference "#PWR0161")
