File: V1/esp-poe-010v-V1.kicad_pcb (KiCad board)
At the start: 4 copper layers, 88 x 45 mm, 95 parts, among them J1 USB_C_Receptacle_USB2.0, J2 RJ45 JACK, J3 1x2P 5,08mm, J4 1x2P 5,08mm, K1 G5NB-1A-E-DC5, K2 G5NB-1A-E-DC5, Q1 UMH3N, Q2 WPM2015-3/TR, Q3 LMUN2211LT1G, Q4 MMBT2222A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

Commit message: dev time
Parts:
- removed C26: 100nF/50V, Tales:C_0402_1005Metric
- removed D10, D9: 1N4148, Tales:D_SOD-123
- removed D7, D8: WHITE, Tales:LED_0603_1608Metric
- removed J3, J4: 1x2P 5,08mm, Tales:TerminalBlock_Dibo_DB142R-5.08-2P_1x02_P5.08mm_Horizontal
- removed K1, K2: G5NB-1A-E-DC5, Tales:Relay_SPST_Omron_G5NB-1A
- removed Q4, Q5: MMBT2222A, Tales:SOT-23
- removed R25, R28: 10k/62,5mW, Tales:R_0402_1005Metric
- removed R26, R29: 1k/62,5mW, Tales:R_0402_1005Metric
- removed R27, R30: 680R/62,5mW, Tales:R_0402_1005Metric
- removed U7: SHT31-DIS, Tales:Sensirion_DFN-8-1EP_2.5x2.5mm_P0.5mm_EP1.1x1.7mm
Routing:
- net +5V: track 109.6 -> 23.5 mm
- net Net-(J3-Pin_1): track 48.6 -> 0.00 mm
- net Net-(J4-Pin_1): track 40.2 -> 0.00 mm
- net I2C_SDA: track 33.5 -> 1.41 mm
- net I2C_SCL: track 33.4 -> 1.39 mm
- net +3.3V: track 139.4 -> 112.9 mm
- net Net-(J3-Pin_2): track 26.0 -> 0.00 mm
- net Net-(J4-Pin_2): track 23.5 -> 0.00 mm
- net GND: track 75.5 -> 61.2 mm, vias 39 -> 36
- net OUT1: track 28.8 -> 17.2 mm, vias 2 -> 1
- net Net-(D10-A): track 7.11 -> 0.00 mm
- net Net-(D7-K): track 7.11 -> 0.00 mm
- net OUT2: track 30.3 -> 26.1 mm, vias 2 -> 1
- net Net-(D8-A): track 1.70 -> 0.00 mm
- net Net-(D7-A): track 1.70 -> 0.00 mm
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Other:
- outline, holes or cut-outs redrawn
- board text added: "ESP-POE-010V V1.0"
- board text removed: "ESP-POE-2RL V1.3"
- board text removed: "OUT1"
- board text removed: "OUT2"
