File: V1/esp-poe-010v-V1.kicad_sch (KiCad schematic)
At the start: 63 parts, among them J1 USB_C_Receptacle_USB2.0, J2 RJ45 JACK, J3 1x2P 5,08mm, J4 1x2P 5,08mm, K1 G5NB-1A-E-DC5, K2 G5NB-1A-E-DC5, Q1 UMH3N, Q2 WPM2015-3/TR, Q3 LMUN2211LT1G, Q4 MMBT2222A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

Commit message: dev time
Parts:
- removed C26: 100nF/50V, Tales:C_0402_1005Metric, symbol Device:C_Small
- removed D10, D9: 1N4148, Tales:D_SOD-123, symbol Diode:1N4148
- removed D7, D8: WHITE, Tales:LED_0603_1608Metric, symbol Device:LED_Small
- removed J3, J4: 1x2P 5,08mm, Tales:TerminalBlock_Dibo_DB142R-5.08-2P_1x02_P5.08mm_Horizontal, symbol Connector_Generic:Conn_01x02
- removed K1, K2: G5NB-1A-E-DC5, Tales:Relay_SPST_Omron_G5NB-1A, symbol Tales:G5NB-1A
- removed Q4, Q5: MMBT2222A, Tales:SOT-23, symbol Transistor_BJT:Q_NPN_BEC
- removed R25, R28: 10k/62,5mW, Tales:R_0402_1005Metric, symbol Device:R_US
- removed R26, R29: 1k/62,5mW, Tales:R_0402_1005Metric, symbol Device:R_US
- removed R27, R30: 680R/62,5mW, Tales:R_0402_1005Metric, symbol Device:R_US
- removed U7: SHT31-DIS, Tales:Sensirion_DFN-8-1EP_2.5x2.5mm_P0.5mm_EP1.1x1.7mm, symbol Sensor_Humidity:SHT31-DIS
- added U7: MCP4728, Package_SO:MSOP-10_3x3mm_P0.5mm, symbol Analog_DAC:MCP4728
Connections:
- no-connect marks 29 -> 27
Other:
- sheet POWER: file esp-poe-2rl-V1-power.kicad_sch -> esp-poe-010v-V1-power.kicad_sch
- note added: "D/A CONVERTER ADDRESS 0x??"
- note added: "ESP32 TEMPLATE FOR GPIO ASSIGNMENT {"NAME":"ESP-POE-010V-V1","GPIO":[0,3200,0,3232,0,0,0,0,5536,224,0,0,225,0,5600,0,0,0,0,5568,0,0,0,0,0,0,0,0,608,640,0,0,0,0,0,0],"FLAG":0,"BASE":1} https://tasmota.github.io/docs/Templates/"
- note removed: "ESP32 TEMPLATE FOR GPIO ASSIGNMENT {"NAME":"ESP-POE-2RL-V1","GPIO":[0,3200,0,3232,0,0,0,0,5536,224,0,0,225,0,5600,0,0,0,0,5568,0,0,0,0,0,0,0,0,608,640,0,0,0,0,0,0],"FLAG":0,"BASE":1} https://tasmota.github.io/docs/Templates/"
- note removed: "TEMP/HUMID ADDRESS 0x44"
- title: ESP 2x Relay Output Module with PoE -> ESP 2x 0-10V Output Module with PoE
