File: V1/eumesmo-io-24v16ch-v6-i2c.kicad_sch (KiCad schematic)
At the start: 26 parts, among them J9 250-203, SW2 1WIRE_SEL, U10 MCP23017, U11 DS2482S-100, U8 MCP23008, U9 MCP23008

Commit message: Development.
Parts:
- removed C26, C28, C30, C33, C35: 100nF/50V, Tales:C_0402_1005Metric, symbol Device:C_Small
- removed C27, C29, C31, C32, C34: 10uF/25V, Tales:C_0805_2012Metric, symbol Device:C_Small
- removed C36: 470pF/50V, Tales:C_0402_1005Metric, symbol Device:C_Small
- removed D8, D9: ESD9L5.0, Diode_SMD:D_SOD-923, symbol Diode:ESD5Zxx
- removed J9: 250-203, Tales:TerminalBlock_Wago_250-203_1x03_P3.5mm_45Degree, symbol Connector_Generic:Conn_01x03
- removed R36, R37, R38: 1k, Tales:R_0402_1005Metric, symbol Device:R_US
- removed R39: 1k8/125mW, Tales:R_0805_2012Metric, symbol Device:R_US
- removed R40: 33R, Tales:R_0402_1005Metric, symbol Device:R_US
- removed SW2: 1WIRE_SEL, Tales:SW_DIP_SPSTx02_Slide_Copal_CHS-02B_W7.62mm_P1.27mm, symbol Switch:SW_DIP_x02
- removed U10: MCP23017, Package_SO:SSOP-28_5.3x10.2mm_P0.65mm, symbol Interface_Expansion:MCP23017x-x-SS
- removed U11: DS2482S-100, Package_SO:SO-8_3.9x4.9mm_P1.27mm, symbol Tales:DS2482-100
- removed U8, U9: MCP23008, Package_SO:SSOP-20_5.3x7.2mm_P0.65mm, symbol Interface_Expansion:MCP23008-xSS
- added U8: ISO1540, Package_SO:SOIC-8_3.9x4.9mm_P1.27mm, symbol Isolator:ISO1540
- added U9: PCA9685PW, Package_SO:TSSOP-28_4.4x9.7mm_P0.65mm, symbol Driver_LED:PCA9685PW
Connections:
- no-connect marks 3 -> 0
Other:
- note removed: "1-WIRE MASTER ADDRESS 0x18"
- note removed: "ATTENTION! DIP SWITCH SW2: ONLY ONE SWITCH CAN BE ON AT ANY GIVEN TIME."
- note removed: "INPUTS ADDRESS 0x20"
- note removed: "INPUTS ADDRESS 0x21"
- note removed: "SENSORS"
