File: V1/eumesmo-io-24v16ch-v6-mcu.kicad_sch (KiCad schematic)
At the start: 19 parts, among them Q3 UMH3N, SW1 RESET, U3 TPS3820-33, U4 CH340K, U5 ESP32-WROOM-32UE-N16

Commit message: Development.
Parts:
- removed R15, R16: 2k2, Tales:R_0402_1005Metric, symbol Device:R_US
Connections:
- net 1WIREGPIO: no longer names the net of U5.27 (IO16)
- net MCPIN1INT: no longer names the net of U5.16 (IO13)
- net MCPIN2INT: no longer names the net of U5.13 (IO14)
- no-connect marks 16 -> 19
