File: V1/eumesmo-io-24v16ch-v6.kicad_sch (KiCad schematic)
At the start: 9 parts, among them J1 250-208, J2 250-208, J3 250-208, J4 250-208, J5 250-202

Commit message: Development.
Parts:
- removed J5: 250-202, Tales:TerminalBlock_Wago_250-202_1x02_P3.5mm_45Degree, symbol Connector_Generic:Conn_01x02
Connections:
- net IN1: no longer names the net of J1.1 (Pin_1)
- net IN10: no longer names the net of J2.2 (Pin_2)
- net IN11: no longer names the net of J2.3 (Pin_3)
- net IN12: no longer names the net of J2.4 (Pin_4)
- net IN13: no longer names the net of J2.5 (Pin_5)
- net IN14: no longer names the net of J2.6 (Pin_6)
- net IN15: no longer names the net of J2.7 (Pin_7)
- net IN16: no longer names the net of J2.8 (Pin_8)
- net IN2: no longer names the net of J1.2 (Pin_2)
- net IN3: no longer names the net of J1.3 (Pin_3)
- net IN4: no longer names the net of J1.4 (Pin_4)
- net IN5: no longer names the net of J1.5 (Pin_5)
- net IN6: no longer names the net of J1.6 (Pin_6)
- net IN7: no longer names the net of J1.7 (Pin_7)
- net IN8: no longer names the net of J1.8 (Pin_8)
- net IN9: no longer names the net of J2.1 (Pin_1)
- net OUT1: no longer names the net of J3.1 (Pin_1)
- net OUT10: no longer names the net of J4.2 (Pin_2)
- net OUT11: no longer names the net of J4.3 (Pin_3)
- net OUT12: no longer names the net of J4.4 (Pin_4)
- net OUT13: no longer names the net of J4.5 (Pin_5)
- net OUT14: no longer names the net of J4.6 (Pin_6)
- net OUT15: no longer names the net of J4.7 (Pin_7)
- net OUT16: no longer names the net of J4.8 (Pin_8)
- net OUT2: no longer names the net of J3.2 (Pin_2)
- net OUT3: no longer names the net of J3.3 (Pin_3)
- net OUT4: no longer names the net of J3.4 (Pin_4)
- net OUT5: no longer names the net of J3.5 (Pin_5)
- net OUT6: no longer names the net of J3.6 (Pin_6)
- net OUT7: no longer names the net of J3.7 (Pin_7)
- net OUT8: no longer names the net of J3.8 (Pin_8)
- net OUT9: no longer names the net of J4.1 (Pin_1)
Other:
- removed sheet Input 1
- removed sheet Input 10
- removed sheet Input 11
- removed sheet Input 12
- removed sheet Input 13
- removed sheet Input 14
- removed sheet Input 15
- removed sheet Input 16
- removed sheet Input 2
- removed sheet Input 3
- removed sheet Input 4
- removed sheet Input 5
- removed sheet Input 6
- removed sheet Input 7
- removed sheet Input 8
- removed sheet Input 9
- removed sheet Output 1
- removed sheet Output 10
- removed sheet Output 11
- removed sheet Output 12
- removed sheet Output 13
- removed sheet Output 14
- removed sheet Output 15
- removed sheet Output 16
- removed sheet Output 2
- removed sheet Output 3
- removed sheet Output 4
- removed sheet Output 5
- removed sheet Output 6
- removed sheet Output 7
- removed sheet Output 8
- removed sheet Output 9
- sheet I2C Devices ports: added none; removed 1WIREGPIO, IN1, IN10, IN11, IN12, IN13, IN14, IN15, IN16, IN2, IN3, IN4, IN5, IN6, IN7, IN8, IN9, MCPIN1INT, MCPIN2INT
- sheet MCU ports: added none; removed 1WIREGPIO, MCPIN1INT, MCPIN2INT
- note added: "OUTPUTS 1-4"
- note added: "OUTPUTS 13-16"
- note added: "OUTPUTS 5-8"
- note added: "OUTPUTS 9-12"
- note removed: "GNDIO"
- note removed: "INPUTS 1-8"
- note removed: "INPUTS 9-16"
- note removed: "OUTPUTS 1-8"
- note removed: "OUTPUTS 9-16"
- moved on the sheet: J1, J2
