File: V1/eumesmo-010-16ch-v1-i2c.kicad_sch (KiCad schematic)
At the start: 4 parts, among them U8 ISO1540, U9 PCA9685PW

Commit message: Restarting fresh
Parts:
- removed U8: ISO1540, Package_SO:SOIC-8_3.9x4.9mm_P1.27mm, symbol Isolator:ISO1540
- removed U9: PCA9685PW, Package_SO:TSSOP-28_4.4x9.7mm_P0.65mm, symbol Driver_LED:PCA9685PW
- added C26, C28, C30, C33, C35: 100nF/50V, Tales:C_0402_1005Metric, symbol Device:C_Small
- added C27, C29, C31, C32, C34: 10uF/25V, Tales:C_0805_2012Metric, symbol Device:C_Small
- added C36: 470pF/50V, Tales:C_0402_1005Metric, symbol Device:C_Small
- added D8, D9: ESD9L5.0, Diode_SMD:D_SOD-923, symbol Diode:ESD5Zxx
- added J9: 250-203, Tales:TerminalBlock_Wago_250-203_1x03_P3.5mm_45Degree, symbol Connector_Generic:Conn_01x03
- added R36, R37, R38: 1k, Tales:R_0402_1005Metric, symbol Device:R_US
- added R39: 1k8/125mW, Tales:R_0805_2012Metric, symbol Device:R_US
- added R40: 33R, Tales:R_0402_1005Metric, symbol Device:R_US
- added SW2: 1WIRE_SEL, Tales:SW_DIP_SPSTx02_Slide_Copal_CHS-02B_W7.62mm_P1.27mm, symbol Switch:SW_DIP_x02
- added U10: MCP23017, Package_SO:SSOP-28_5.3x10.2mm_P0.65mm, symbol Interface_Expansion:MCP23017x-x-SS
- added U11: DS2482S-100, Package_SO:SO-8_3.9x4.9mm_P1.27mm, symbol Tales:DS2482-100
- added U8, U9: MCP23008, Package_SO:SSOP-20_5.3x7.2mm_P0.65mm, symbol Interface_Expansion:MCP23008-xSS
Connections:
- net I2CSCL: now also U10.12 (SCK), U11.4 (SCL), U8.1 (SCL), U9.1 (SCL)
- net I2CSDA: now also U10.13 (SDA), U11.5 (SDA), U8.2 (SDA), U9.2 (SDA)
- new net +3V3: C26.1, C27.1, C28.1, C29.1, C30.1, C31.1, C32.1, C33.1, R36.1, R37.1, R38.1, R39.1, U10.16 (A1), U10.9 (V_{DD}), U11.1 (V_{CC}), U8.20 (VDD), U9.20 (VDD), U9.5 (A0)
- new net +5V: C34.1, C35.1, D8.1 (K), J9.1 (Pin_1)
- new net 1WIREBUS: C36.1, R39.2, R40.2, SW2.1, SW2.2
- new net 1WIREFIELD: D9.1 (K), J9.2 (Pin_2), R40.1
- new net 1WIREGPIO: SW2.3
- new net 1WIREMASTER: SW2.4, U11.2 (IO)
- new net GND: C26.2, C27.2, C28.2, C29.2, C30.2, C31.2, C32.2, C33.2, C34.2, C35.2, C36.2, D8.2 (A), D9.2 (A), J9.3 (Pin_3), U10.10 (V_{SS}), U10.15 (A0), U10.17 (A2), U11.3 (GND), U11.7 (AD1), U11.8 (AD0), U8.3 (A2), U8.4 (A1), U8.5 (A0), U8.9 (VSS), U9.3 (A2), U9.4 (A1), U9.9 (VSS)
- new net IN1: U8.12 (GP0)
- new net IN10: U9.13 (GP1)
- new net IN11: U9.14 (GP2)
- new net IN12: U9.15 (GP3)
- new net IN13: U9.16 (GP4)
- new net IN14: U9.17 (GP5)
- new net IN15: U9.18 (GP6)
- new net IN16: U9.19 (GP7)
- new net IN2: U8.13 (GP1)
- new net IN3: U8.14 (GP2)
- new net IN4: U8.15 (GP3)
- new net IN5: U8.16 (GP4)
- new net IN6: U8.17 (GP5)
- new net IN7: U8.18 (GP6)
- new net IN8: U8.19 (GP7)
- new net IN9: U9.12 (GP0)
- new net MCPIN1INT: U8.8 (INT)
- new net MCPIN2INT: U9.8 (INT)
- new net MCPINN1RST: R36.2, U8.6 (~{RESET})
- new net MCPINN2RST: R37.2, U9.6 (~{RESET})
- new net MCPOUTNRST: R38.2, U10.18 (~{RESET})
- new net OUT1: U10.21 (GPA0)
- new net OUT10: U10.2 (GPB1)
- new net OUT11: U10.3 (GPB2)
- new net OUT12: U10.4 (GPB3)
- new net OUT13: U10.5 (GPB4)
- new net OUT14: U10.6 (GPB5)
- new net OUT15: U10.7 (GPB6)
- new net OUT16: U10.8 (GPB7)
- new net OUT2: U10.22 (GPA1)
- new net OUT3: U10.23 (GPA2)
- new net OUT4: U10.24 (GPA3)
- new net OUT5: U10.25 (GPA4)
- new net OUT6: U10.26 (GPA5)
- new net OUT7: U10.27 (GPA6)
- new net OUT8: U10.28 (GPA7)
- new net OUT9: U10.1 (GPB0)
- no-connect marks 0 -> 3
Other:
- note added: "1-WIRE MASTER ADDRESS 0x18"
- note added: "ATTENTION! DIP SWITCH SW2: ONLY ONE SWITCH CAN BE ON AT ANY GIVEN TIME."
- note added: "INPUTS ADDRESS 0x20"
- note added: "INPUTS ADDRESS 0x21"
- note added: "SENSORS"

Commit message: Development
Parts:
- removed C26, C28, C33, C35: 100nF/50V, Tales:C_0402_1005Metric, symbol Device:C_Small
- removed C27, C29, C32, C34: 10uF/25V, Tales:C_0805_2012Metric, symbol Device:C_Small
- removed C36: 470pF/50V, Tales:C_0402_1005Metric, symbol Device:C_Small
- removed D8, D9: ESD9L5.0, Diode_SMD:D_SOD-923, symbol Diode:ESD5Zxx
- removed J9: 250-203, Tales:TerminalBlock_Wago_250-203_1x03_P3.5mm_45Degree, symbol Connector_Generic:Conn_01x03
- removed R36, R37: 1k, Tales:R_0402_1005Metric, symbol Device:R_US
- removed SW2: 1WIRE_SEL, Tales:SW_DIP_SPSTx02_Slide_Copal_CHS-02B_W7.62mm_P1.27mm, symbol Switch:SW_DIP_x02
- removed U11: DS2482S-100, Package_SO:SO-8_3.9x4.9mm_P1.27mm, symbol Tales:DS2482-100
- removed U8, U9: MCP23008, Package_SO:SSOP-20_5.3x7.2mm_P0.65mm, symbol Interface_Expansion:MCP23008-xSS
- added D10, D11, D12, D13, D14, D15, D16, D17, D18, D19, D20, D21, D22, D23, D8, D9: WHITE/0603, Tales:LED_0603_1608Metric, symbol Device:LED_Small
- added R41, R42, R43, R44, R45, R46, R47, R48, R49, R50, R51, R52, R53, R54: 510R, Tales:R_0402_1005Metric, symbol Device:R_US
- R39: value 1k8/125mW -> 510R; footprint Tales:R_0805_2012Metric -> Tales:R_0402_1005Metric; Case 0805/2012 -> 0402/1005; LCSC Part # C17398 -> C25123; Mfr PN 0805W8F1801T5E -> 0402WGF5100TCE; Vendor PN C17398 -> C25123
- R40: value 33R -> 510R; LCSC Part # C25105 -> C25123; Mfr PN 0402WGF330JTCE -> 0402WGF5100TCE; Vendor PN C25105 -> C25123
Connections:
- net +3V3: no longer R39.1
- net 1WIREBUS: no longer names the net of R40.2
- net 1WIREBUS: no longer R39.2
- net 1WIREFIELD: no longer names the net of R40.1
- net 1WIREFIELD: now also D9.2 (A)
- net OUT1: no longer names the net of U10.21 (GPA0)
- net OUT10: no longer names the net of U10.2 (GPB1)
- net OUT11: no longer names the net of U10.3 (GPB2)
- net OUT12: no longer names the net of U10.4 (GPB3)
- net OUT13: no longer names the net of U10.5 (GPB4)
- net OUT14: no longer names the net of U10.6 (GPB5)
- net OUT15: no longer names the net of U10.7 (GPB6)
- net OUT16: no longer names the net of U10.8 (GPB7)
- net OUT2: no longer names the net of U10.22 (GPA1)
- net OUT3: no longer names the net of U10.23 (GPA2)
- net OUT4: no longer names the net of U10.24 (GPA3)
- net OUT5: no longer names the net of U10.25 (GPA4)
- net OUT6: no longer names the net of U10.26 (GPA5)
- net OUT7: no longer names the net of U10.27 (GPA6)
- net OUT8: no longer names the net of U10.28 (GPA7)
- net OUT9: no longer names the net of U10.1 (GPB0)
- new net: D10.2 (A), R41.1
- new net: D13.2 (A), R44.1
- new net: D19.2 (A), R50.1
- new net: D23.2 (A), R54.1
- new net: D22.2 (A), R53.1
- new net: D12.2 (A), R43.1
- new net: D11.2 (A), R42.1
- new net: D17.2 (A), R48.1
- new net: D16.2 (A), R47.1
- new net: D20.2 (A), R51.1
- new net: D8.2 (A), R39.1
- new net: D14.2 (A), R45.1
- new net: D18.2 (A), R49.1
- new net: D15.2 (A), R46.1
- new net: D21.2 (A), R52.1
- no-connect marks 3 -> 2
Other:
- note removed: "1-WIRE MASTER ADDRESS 0x18"
- note removed: "ATTENTION! DIP SWITCH SW2: ONLY ONE SWITCH CAN BE ON AT ANY GIVEN TIME."
- note removed: "INPUTS ADDRESS 0x20"
- note removed: "INPUTS ADDRESS 0x21"
- note removed: "SENSORS"
- moved on the sheet: C30, C31, R38, TP16, TP17, U10

Commit message: Development
Parts:
- added U8: PCA9685PW, Package_SO:TSSOP-28_4.4x9.7mm_P0.65mm, symbol Driver_LED:PCA9685PW
- U10: Technology (none) -> I/O Expander
Connections:
- net +3V3: now also R39.2, R40.2, R41.2, R42.2, R43.2, R44.2, R45.2, R46.2, R47.2, R48.2, R49.2, R50.2, R51.2, R52.2, R53.2, R54.2
- net at D9.1 (K): now also U10.22 (GPA1)
- net at D13.1 (K): now also U10.26 (GPA5)
- net at D23.1 (K): now also U10.8 (GPB7)
- net at D22.1 (K): now also U10.7 (GPB6)
- net at D17.1 (K): now also U10.2 (GPB1)
- net at D20.1 (K): now also U10.5 (GPB4)
- net at D8.1 (K): now also U10.21 (GPA0)
- net at D10.1 (K): now also U10.23 (GPA2)
- net at D18.1 (K): now also U10.3 (GPB2)
- net at D15.1 (K): now also U10.28 (GPA7)
- net at D11.1 (K): now also U10.24 (GPA3)
- net at D16.1 (K): now also U10.1 (GPB0)
- net at U10.25 (GPA4): now also D12.1 (K)
- net at U10.27 (GPA6): now also D14.1 (K)
- net at U10.4 (GPB3): now also D19.1 (K)
- net at U10.6 (GPB5): now also D21.1 (K)
Other:
- moved on the sheet: C30, C31, D10, D11, D12, D13, D14, D15, D16, D17, D18, D19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

Commit message: Development
Parts:
- added R36, R37: 2k2, Tales:R_0402_1005Metric, symbol Device:R_US
- added U13: ISO1540, Package_SO:SOIC-8_3.9x4.9mm_P1.27mm, symbol Isolator:ISO1540
Connections:
- net GND: now also U13.4 (GND1)
- net I2CSCL: now also U13.3 (SCL1)
- net I2CSDA: now also U13.2 (SDA1)
- net GNDA: now reaches U8.1 (A0)
- net GNDA: now also U8.14 (VSS), U8.2 (A1), U8.23 (~{OE}), U8.24 (A5), U8.25 (EXTCLK), U8.3 (A2), U8.4 (A3), U8.5 (A4), U13.5 (GND2)
- net at U8.26 (SCL): now also R36.2, U13.6 (SCL2)
- net at U8.27 (SDA): now also R37.2, U13.7 (SDA2)
- net +5VA: now reaches U8.28 (VDD)
- net +5VA: now also R36.1, R37.1, U13.8 (VCC2)
- new net +5V: U13.1 (VCC1)
Other:
- moved on the sheet: C30, C31, D10, D11, D12, D13, D14, D15, D16, D17, D18, D19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

Commit message: Development
Parts:
- added C34, C35, C36, C37, C38, C39, C40, C41, C42, C43, C44, C45, C46, C47, C48, C49: 1uF/50V, Tales:C_0805_2012Metric, symbol Device:C_Small
- added C50, C51, C52, C53: 100nF/50V, Tales:C_0402_1005Metric, symbol Device:C_Small
- added R100, R15, R16, R55, R56, R57, R58, R59, R60, R61, R62, R63, R64, R65, R66, R67, R68, R69, R70, R71, R72, R73, R74, R75, R76, R77, R78, R79, R80, R81, R82, R83, R84, R85, R86, R87, R88, R89, R90, R91, R92, R93, R94, R95, R96, R97, R98, R99: 10k, Tales:R_0402_1005Metric, symbol Device:R_US
- added R101, R102, R103, R104, R105, R106, R107, R108, R109, R110, R111, R112, R113, R114, R115, R116: 47R, Tales:R_0805_2012Metric, symbol Device:R_US
- added U14, U15, U16, U17: LM324, symbol Amplifier_Operational:LM324
Connections:
- net +3V3: no longer U10.16 (A1)
- net GND: now also U10.16 (A1)
- net GNDA: now also C34.2, C35.2, C36.2, C37.2, C38.2, C39.2, C40.2, C41.2, C42.2, C43.2, C44.2, C45.2, C46.2, C47.2, C48.2, C49.2, C50.2, C51.2, C52.2, C53.2, R100.1, R55.1, R58.1, R61.1, R64.1, R70.1, R72.1, R74.1, R76.1, R82.1, R84.1, R86.1, R88.1, R94.1, R96.1, R98.1, U14.11 (V-), U15.11 (V-), U16.11 (V-), U17.11 (V-)
- net PWM05: now reaches U8.10 (LED4)
- net PWM05: now also R65.1
- net PWM06: now reaches U8.11 (LED5)
- net PWM06: now also R66.1
- net PWM07: now reaches U8.12 (LED6)
- net PWM07: now also R67.1
- net PWM08: now reaches U8.13 (LED7)
- net PWM08: now also R68.1
- net PWM09: now reaches U8.15 (LED8)
- net PWM09: now also R77.1
- net PWM10: now reaches U8.16 (LED9)
- net PWM10: now also R78.1
- net PWM11: now reaches U8.17 (LED10)
- net PWM11: now also R79.1
- net PWM12: now reaches U8.18 (LED11)
- net PWM12: now also R80.1
- net PWM13: now reaches U8.19 (LED12)
- net PWM13: now also R89.1
- net PWM14: now reaches U8.20 (LED13)
- net PWM14: now also R90.1
- net PWM15: now reaches U8.21 (LED14)
- net PWM15: now also R91.1
- net PWM16: now reaches U8.22 (LED15)
- net PWM16: now also R92.1
- net PWM01: now reaches U8.6 (LED0)
- net PWM01: now also R15.1
- net PWM02: now reaches U8.7 (LED1)
- net PWM02: now also R56.1
- net PWM03: now reaches U8.8 (LED2)
- net PWM03: now also R59.1
- net PWM04: now reaches U8.9 (LED3)
- net PWM04: now also R62.1
- new net: C46.1, R89.2, U17.3 (+)
- new net: C49.1, R92.2, U17.12 (+)
- new net: R100.2, R99.1, U17.13 (-)
- new net: R116.1, R99.2, U17.14
- new net: R87.1, R88.2, U16.13 (-)
- new net: R112.1, R87.2, U16.14
- new net: C45.1, R80.2, U16.12 (+)
- new net: C48.1, R91.2, U17.10 (+)
- new net: R102.1, R57.2, U14.7
- new net: C36.1, R59.2, U14.10 (+)
- new net: R73.1, R74.2, U15.9 (-)
- new net: R107.1, R73.2, U15.8
- new net: R104.1, R63.2, U14.14
- new net: C44.1, R79.2, U16.10 (+)
- new net: R60.1, R61.2, U14.9 (-)
- new net: R75.1, R76.2, U15.13 (-)
- new net: R108.1, R75.2, U15.14
- new net: R97.1, R98.2, U17.9 (-)
- new net: R115.1, R97.2, U17.8
- new net: R85.1, R86.2, U16.9 (-)
- new net: R111.1, R85.2, U16.8
- new net: R71.1, R72.2, U15.6 (-)
- new net: R81.1, R82.2, U16.2 (-)
- new net: R109.1, R81.2, U16.1
- new net: C35.1, R56.2, U14.5 (+)
- new net: C38.1, R65.2, U15.3 (+)
- new net: C34.1, R15.2, U14.3 (+)
- new net: C37.1, R62.2, U14.12 (+)
- new net: C41.1, R68.2, U15.12 (+)
- new net: C43.1, R78.2, U16.5 (+)
- new net: R83.1, R84.2, U16.6 (-)
- new net: R110.1, R83.2, U16.7
- new net: C40.1, R67.2, U15.10 (+)
- new net: R93.1, R94.2, U17.2 (-)
- new net: R57.1, R58.2, U14.6 (-)
- new net: R103.1, R60.2, U14.8
- new net: R69.1, R70.2, U15.2 (-)
- new net: C39.1, R66.2, U15.5 (+)
- new net: R106.1, R71.2, U15.7
- new net: R105.1, R69.2, U15.1
- new net: R63.1, R64.2, U14.13 (-)
- new net: C42.1, R77.2, U16.3 (+)
- new net: R95.1, R96.2, U17.6 (-)
- new net: R114.1, R95.2, U17.7
- new net: R101.1, R16.2, U14.1
- new net: R16.1, R55.2, U14.2 (-)
- new net: R113.1, R93.2, U17.1
- new net: C47.1, R90.2, U17.5 (+)
- new net +12VA: C50.1, C51.1, C52.1, C53.1, U14.4 (V+), U15.4 (V+), U16.4 (V+), U17.4 (V+)
- new net CH01: R101.2
- new net CH02: R102.2
- new net CH03: R103.2
- new net CH04: R104.2
- new net CH05: R105.2
- new net CH06: R106.2
- new net CH07: R107.2
- new net CH08: R108.2
- new net CH09: R109.2
- new net CH10: R110.2
- new net CH11: R111.2
- new net CH12: R112.2
- new net CH13: R113.2
- new net CH14: R114.2
- new net CH15: R115.2
- new net CH16: R116.2
Other:
- note added: "OUTPUTS ADDRESS 0x20"
- note added: "PWM ADDRESS 0x40"
- note removed: "OUTPUTS ADDRESS 0x22"
- moved on the sheet: C30, C31, D10, D11, D12, D13, D14, D15, D16, D17, D18, D19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

Commit message: Development
Parts:
- added C54, C55, C56: 100nF/50V, Tales:C_0402_1005Metric, symbol Device:C_Small
Connections:
- net +5V: now also C54.1
- net +5VA: now also C55.1, C56.1
- net GNDA: now also C54.2, C55.2, C56.2
Other:
- moved on the sheet: R36, R37, TP16, TP17, U13, U8

Commit message: Development
Parts:
- removed C31: 10uF/25V, Tales:C_0805_2012Metric, symbol Device:C_Small
