File: V1/eumesmo-010-16ch-v1-i2c.kicad_sch (KiCad schematic)
At the start: 42 parts, among them U10 ISO1540, U11 PCA9685PW, U12 MCP23017

Commit message: Adjusted components according to availability in JLCPCB.
Parts:
- C29, C30, C31, C32, D10, D11, D12, D13, D14, D15, D16, D17, D18, D19, D20, D21, D22, D23, D24, D9, R44, U10, U11, U12: JLCPCB BOM 1 -> (none)
- R35, R36, R37, R38, R39, R42, R43, R45, R46, R47, R48, R49, R50, R51, R52, R53: value 300R -> 330R; JLCPCB BOM 1 -> (none); LCSC Part # C25102 -> C25104; Mfr PN 0402WGF3000TCE -> 0402WGF3300TCE; Vendor PN C25102 -> C25104
- R40, R41: value 2k2 -> 2,2k; JLCPCB BOM 1 -> (none)

Commit message: Text translated to english
Other:
- note added: "PCA9685 MUST BE CONFIGURED FOR PWM FREQUENCY OF 1526 Hz."
- note removed: "PCA9685 DEVE SER CONFIGURADO PARA FREQUÊNCIA PWM DE 1526 Hz."
Changed lines of the file:
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@@
 		)
 	)
-	(text "PCA9685 DEVE SER CONFIGURADO\nPARA FREQUÊNCIA PWM DE 1526 Hz."
+	(text "PCA9685 MUST BE CONFIGURED\nFOR PWM FREQUENCY OF 1526 Hz."
 		(exclude_from_sim no)
 		(at 321.31 191.77 0)
