File: V1/eumesmo-010-16ch-v1-mcu.kicad_sch (KiCad schematic)
At the start: 18 parts, among them Q3 UMH3N, SW1 RESET, U5 TPS3820-33, U6 CH340K, U7 ESP32-WROOM-32UE-N16

Commit message: Development
Parts:
- removed TP11: D+, TestPoint:TestPoint_Pad_D1.5mm, symbol Connector:TestPoint
- removed TP12: D-, TestPoint:TestPoint_Pad_D1.5mm, symbol Connector:TestPoint
- renumbered D24 to D7, R133 to R15, R15 to R16, R16 to R17, R17 to R18, R18 to R19
Other:
- title: eumesmo 24V 16xIn/16xOut/1-Wire Module -> eumesmo 24V 16x 0-10V module
