File: V1/eumesmo-010-16ch-v1-mcu.kicad_sch (KiCad schematic)
At the start: 16 parts, among them Q3 UMH3N, SW1 RESET, U5 TPS3820-33, U6 CH340K, U7 ESP32-WROOM-32UE-N16

Commit message: Adjusted components according to availability in JLCPCB.
Parts:
- C19, C20, C21, D7, Q3, R13, R14, R16, R17, SW1, U5, U6, U7: JLCPCB BOM 1 -> (none)
- R15: value 300R -> 330R; JLCPCB BOM 1 -> (none); LCSC Part # C25102 -> C25104; Mfr PN 0402WGF3000TCE -> 0402WGF3300TCE; Vendor PN C25102 -> C25104
- R18, R19: value 2k2 -> 2,2k; JLCPCB BOM 1 -> (none)
Changed lines of the file:
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@@
 			)
 		)
-		(property "JLCPCB BOM" "1"
-			(at 215.9 93.98 90)
-			(hide yes)
-			(show_name no)
-			(do_not_autoplace no)
-			(effects
-				(font
-					(size 1.27 1.27)
-				)
-			)
-		)
 		(pin "2"
 		)
@@
 			)
 		)
-		(property "JLCPCB BOM" "1"
-			(at 160.02 53.34 0)
-			(hide yes)
-			(show_name no)
-			(do_not_autoplace no)
-			(effects
-				(font
-					(size 1.27 1.27)
-				)
-			)
-		)
 		(property "LCSC Part #" "C15850"
 			(at 162.56 58.4138 0)
@@
 			)
 		)
-		(property "JLCPCB BOM" "1"
-			(at 123.19 55.88 0)
-			(hide yes)
-			(show_name no)
-			(do_not_autoplace no)
-			(effects
-				(font
-					(size 1.27 1.27)
-				)
-			)
-		)
 		(property "Package" ""
 			(at 123.19 55.88 0)
@@
 			)
 		)
-		(property "JLCPCB BOM" "1"
-			(at 209.55 58.42 0)
-			(hide yes)
-			(show_name no)
-			(do_not_autoplace no)
-			(effects
-				(font
-					(size 1.27 1.27)
-				)
-			)
-		)
 		(property "Package" ""
 			(at 209.55 58.42 0)
@@
 			)
 		)
-		(property "JLCPCB BOM" "1"
-			(at 182.88 53.34 0)
-			(hide yes)
-			(show_name no)
-			(do_not_autoplace no)
-			(effects
-				(font
-					(size 1.27 1.27)
-				)
-			)
-		)
 		(property "LCSC Part #" "C307331"
 			(at 185.42 58.4138 0)
@@
 			)
 		)
-		(property "JLCPCB BOM" "1"
-			(at 106.68 59.69 0)
-			(hide yes)
-			(show_name no)
-			(do_not_autoplace no)
-			(effects
-				(font
-					(size 1.27 1.27)
-				)
-			)
-		)
 		(property "LCSC Part #" "C62892"
 			(at 110.49 63.5 0)
@@
 			)
 		)
-		(property "JLCPCB BOM" "1"
-			(at 106.68 80.01 0)
-			(hide yes)
-			(show_name no)
-			(do_not_autoplace no)
-			(effects
-				(font
-					(size 1.27 1.27)
-				)
-			)
-		)
 		(property "LCSC Part #" "C62892"
 			(at 110.49 83.82 0)
@@
 			)
 		)
-		(property "Value" "2k2"
+		(property "Value" "2,2k"
 			(at 262.89 109.22 0)
 			(show_name no)
@@
 			)
 		)
-		(property "JLCPCB BOM" "1"
-			(at 260.35 109.22 0)
-			(hide yes)
-			(show_name no)
-			(do_not_autoplace no)
-			(effects
-				(font
-					(size 1.27 1.27)
-				)
-			)
-		)
 		(pin "1"
 		)
@@
 			)
 		)
-		(property "JLCPCB BOM" "1"
-			(at 123.19 97.79 0)
-			(hide yes)
-			(show_name no)
-			(do_not_autoplace no)
-			(effects
-				(font
-					(size 1.27 1.27)
-				)
-			)
-		)
 		(property "LCSC Part #" "C720477"
 			(at 127 100.3301 90)
@@
 			)
 		)
-		(property "Value" "300R"
+		(property "Value" "330R"
 			(at 232.41 64.77 90)
 			(show_name no)
@@
 			)
 		)
-		(property "Mfr PN" "0402WGF3000TCE"
+		(property "Mfr PN" "0402WGF3300TCE"
 			(at 232.41 71.12 0)
 			(hide yes)
@@
 			)
 		)
-		(property "Vendor PN" "C25102"
+		(property "Vendor PN" "C25104"
 			(at 232.41 71.12 0)
 			(hide yes)
@@
 			)
 		)
-		(property "LCSC Part #" "C25102"
+		(property "LCSC Part #" "C25104"
 			(at 232.41 67.31 90)
 			(show_name no)
@@
 			)
 		)
-		(property "JLCPCB BOM" "1"
-			(at 232.41 71.12 0)
-			(hide yes)
-			(show_name no)
-			(do_not_autoplace no)
-			(effects
-				(font
-					(size 1.27 1.27)
-				)
-			)
-		)
 		(pin "1"
 		)
@@
 			)
 		)
-		(property "JLCPCB BOM" "1"
-			(at 246.38 87.63 0)
-			(hide yes)
-			(show_name no)
-			(do_not_autoplace no)
-			(effects
-				(font
-					(size 1.27 1.27)
-				)
-			)
-		)
 		(property "Package" ""
 			(at 246.38 87.63 0)
@@
 			)
 		)
-		(property "Value" "2k2"
+		(property "Value" "2,2k"
 			(at 248.92 109.22 0)
 			(show_name no)
@@
 			)
 		)
-		(property "JLCPCB BOM" "1"
-			(at 246.38 109.22 0)
-			(hide yes)
-			(show_name no)
-			(do_not_autoplace no)
-			(effects
-				(font
-					(size 1.27 1.27)
-				)
-			)
-		)
 		(pin "1"
 		)
@@
 			)
 		)
-		(property "JLCPCB BOM" "1"
-			(at 179.07 96.52 0)
-			(hide yes)
-			(show_name no)
-			(do_not_autoplace no)
-			(effects
-				(font
-					(size 1.27 1.27)
-				)
-			)
-		)
 		(property "LCSC Part #" "C701346"
 			(at 182.88 137.16 0)
@@
 			)
 		)
-		(property "JLCPCB BOM" "1"
-			(at 250.19 71.12 0)
-			(hide yes)
-			(show_name no)
-			(do_not_autoplace no)
-			(effects
-				(font
-					(size 1.27 1.27)
-				)
-			)
-		)
-		(property "Sim.Pin" "1=K 2=A"
-			(at 250.19 71.12 0)
-			(hide yes)
-			(show_name no)
-			(do_not_autoplace no)
-			(effects
-				(font
-					(size 1.27 1.27)
-				)
-			)
-		)
-		(property "Sim.Pins" "1=K 2=A"
-			(at 250.19 71.12 0)
-			(hide yes)
-			(show_name no)
-			(do_not_autoplace no)
-			(effects
-				(font
-					(size 1.27 1.27)
-				)
-			)
-		)
 		(pin "1"
 		)
@@
 			)
 		)
-		(property "JLCPCB BOM" "1"
-			(at 143.51 66.04 0)
-			(hide yes)
-			(show_name no)
-			(do_not_autoplace no)
-			(effects
-				(font
-					(size 1.27 1.27)
-				)
-			)
-		)
 		(property "LCSC Part #" "C130064"
 			(at 146.05 78.74 0)
@@
 			)
 		)
-		(property "JLCPCB BOM" "1"
-			(at 63.5 72.39 0)
-			(hide yes)
-			(show_name no)
-			(do_not_autoplace no)
-			(effects
-				(font
-					(size 1.27 1.27)
-				)
-			)
-		)
 		(property "LCSC Part #" "C968586"
 			(at 66.04 92.71 0)
@@
 			(at 43.18 48.26 0)
 			(hide yes)
-			(show_name no)
-			(do_not_autoplace no)
-			(effects
-				(font
-					(size 1.27 1.27)
-				)
-			)
-		)
-		(property "JLCPCB BOM" "1"
-			(at 43.18 48.26 0)
-			(hide yes)
