File: V1/eumesmo-010-16ch-v1-mcu.kicad_sch (KiCad schematic)
At the start: 16 parts, among them Q3 UMH3N, SW1 RESET, U5 TPS3820-33, U6 CH340K, U7 ESP32-WROOM-32UE-N16

Commit message: Change LEDs for orange
Parts:
- D7: value WHITE/0603 -> ORANGE/0603; LCSC Part # C2290 -> C2987557; Mfr Hubei KENTO Elec -> Everlight Elec; Mfr PN KT-0603W -> 19-217/S2C-AL1M2VY/6T; Vendor PN C2290 -> C2987557
- R15: value 330R -> 680R; FT Rotation Offset (none) -> 0; LCSC Part # C25104 -> C25130; Mfr PN 0402WGF3300TCE -> 0402WGF6800TCE; Vendor PN C25104 -> C25130

Commit message: Component rotations and offsets ajusted for JLCPCB
Parts:
- R15: FT Rotation Offset 0 -> (none)
Changed lines of the file:
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@@
 			)
 		)
-		(property "FT Rotation Offset" "0"
+		(property "FT Rotation Offset" ""
 			(at 232.41 71.12 90)
 			(hide yes)
