File: V1/eumesmo-010-16ch-v1-power.kicad_sch (KiCad schematic)
At the start: 51 parts, among them J6 250-202, J7 USB_C_Receptacle_USB2.0, Q1 WPM2015-3/TR, Q2 MMUN2211LT3G, U1 TX4138, U2 SY8089A1AAC

Commit message: Restarting fresh
Other:
- moved on the sheet: C10, C11, C12, C13, C14, C6, C7, C8, C9, D4, D5, D6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

Commit message: Development
Parts:
- added C26: 1uF/50V, Tales:C_0805_2012Metric, symbol Device:C_Small
- added C27: 10uF/25V, Tales:C_0805_2012Metric, symbol Device:C_Small
- added U11: L78L12, Package_TO_SOT_SMD:SOT-89-3, symbol Regulator_Linear:L78L12_SOT89
- added U12: L78L05, Package_TO_SOT_SMD:SOT-89-3, symbol Regulator_Linear:L78L05_SOT89
- added U9: B2415S-1WR3, symbol Tales:B2415S-1WR3
Connections:
- net +24V: now also C26.1, U9.2 (Vin)
- net GND: now also C26.2, U9.1 (GND)
- new net +12VA: U11.1 (OUT)
- new net +15VA: C27.1, U11.3 (IN), U12.3 (IN), U9.4 (Vout)
- new net +5VA: U12.1 (OUT)
- new net GNDA: C27.2, U11.2 (GND), U12.2 (GND), U9.3 (0V)
Other:
- moved on the sheet: C10, C11, C12, C13, C14, C2, C3, C6, C7, C8, C9, D4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

Commit message: Development
Parts:
- added C28, C32: 1uF/50V, Tales:C_0805_2012Metric, symbol Device:C_Small
- added C29, C33: 100nF/50V, Tales:C_0402_1005Metric, symbol Device:C_Small
Connections:
- net +12VA: now also U12.3 (IN), C28.1, C29.1
- net +5VA: now also C32.1, C33.1
- net GNDA: now also C28.2, C29.2, C32.2, C33.2
- net +15VA: no longer names the net of C27.1, U11.3 (IN), U9.4 (Vout)
- net +15VA: no longer U12.3 (IN)
Other:
- note added: "ANALOG POWER RAILS"
- moved on the sheet: C26, C27, U11, U12, U9

Commit message: Development
Parts:
- removed C6: 1uF/50V, Tales:C_0805_2012Metric, symbol Device:C_Small
- added C31: 10uF/25V, Tales:C_0805_2012Metric, symbol Device:C_Small
Connections:
- net 5VUSB: now also C31.1
- net GND: now also C31.2

Commit message: Development
Parts:
- removed C27: 10uF/25V, Tales:C_0805_2012Metric, symbol Device:C_Small
- removed C28: 1uF/50V, Tales:C_0805_2012Metric, symbol Device:C_Small
- removed C29: 100nF/50V, Tales:C_0402_1005Metric, symbol Device:C_Small
- removed U11: L78L12, Package_TO_SOT_SMD:SOT-89-3, symbol Regulator_Linear:L78L12_SOT89
- removed U12: L78L05, Package_TO_SOT_SMD:SOT-89-3, symbol Regulator_Linear:L78L05_SOT89
- removed U9: B2415S-1WR3, symbol Tales:B2415S-1WR3
- added C7: 10uF/25V, Tales:C_0805_2012Metric, symbol Device:C_Small
- added U2: L78L05_SOT89, Package_TO_SOT_SMD:SOT-89-3, symbol Regulator_Linear:L78L05_SOT89
- added U3: B2412S-1WR3, Tales:Ylptec BxxxxS-1WR3, symbol Tales:B2412S-1WR3
- D6: Technology (none) -> LED
- renumbered C31 to C10, C7 to C11, C8 to C12, C9 to C13, C10 to C14, C11 to C15, C12 to C16, C13 to C17, C14 to C18, C26 to C6, C32 to C8, C33 to C9, J6 to J5, J7 to J6, TP9 to TP10, TP7 to TP6, TP6 to TP7, TP10 to TP9, U2 to U4
Connections:
- net +12VA: now also C7.1, U2.3 (IN), U3.4 (Vout)
- net +24V: now also U3.2 (Vin)
- net +5VA: now also U2.1 (OUT)
- net GND: now also U3.1 (GND)
- net GNDA: now also C7.2, U2.2 (GND), U3.3 (0V)
Other:
- moved on the sheet: C6, C8, C9

Commit message: Development
Parts:
- R11: value 1k -> 300R; LCSC Part # C11702 -> C25102; Mfr PN 0402WGF1001TCE -> 0402WGF3000TCE; Vendor PN C11702 -> C25102
Connections:
- net +3V3: now also R11.1
- net +5V: no longer R11.1
- net USBCD+: now also D5.1 (I/O1); no longer D5.3 (I/O2)
- net USBCD-: now also D5.3 (I/O2); no longer D5.1 (I/O1)
- net USBD+: now also D5.6 (I/O1); no longer D5.4 (I/O2)
- net USBD-: now also D5.4 (I/O2); no longer D5.6 (I/O1)
- net 5VLED renamed 3V3LED
Other:
- note added: "V_{F} = 2.68V @2.0mA R_{LED} = (3.3V - 2.68V) / 2.0mA R_{LED} = 0.62 / 0.002 R_{LED} = 310 ohm USE C25102 300R -> 2.07mA"
- note removed: "I_{LED} = (5V - V_{LED}) / 1k I_{LED} = (5V - 2.7V) / 1k I_{LED} = 2,30 mA"
- moved on the sheet: C16, C17, C18, D6, L3, R10, R11, R12, TP10, U4
