File: V1/eumesmo-010-16ch-v1-power.kicad_sch (KiCad schematic)
At the start: 57 parts, among them J5 250-202, J6 USB_C_Receptacle_USB2.0, Q1 WPM2015-3/TR, Q2 MMUN2211LT3G, U1 TX4138, U2 L78L05_SOT89, U3 B2412S-1WR3, U4 SY8089A1AAC

Commit message: Development
Parts:
- removed TP4, TP5: GND, Tales:TestPoint_Keystone_5019_Miniature, symbol Connector:TestPoint
Other:
- moved on the sheet: R5

Commit message: Development
Parts:
- renumbered TP6 to TP4, TP7 to TP5, TP8 to TP6, TP9 to TP7, TP10 to TP8
Other:
- title: eumesmo 24V 16xIn/16xOut/1-Wire Module -> eumesmo 24V 16x 0-10V module
Changed lines of the file:
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@@
 	(paper "A4")
 	(title_block
-		(title "eumesmo 24V 16xIn/16xOut/1-Wire Module")
-		(date "2026-06-17")
-		(rev "V6.2")
+		(title "eumesmo 24V 16x 0-10V module")
+		(date "2026-06-23")
+		(rev "V1.0")
 	)
 	(text "RESISTORS: 62,5mW WHERE NOT SPECIFIED"
@@
 		(in_pos_files yes)
 		(dnp yes)
-		(property "Reference" "TP8"
+		(property "Reference" "TP6"
 			(at 154.94 125.73 0)
 			(show_name no)
@@
 			(project "eumesmo-010-16ch-v1"
 				(path "/2bc5a21a-1d79-419d-a592-6852cc07b00a/7b388c9c-6faf-4681-b727-510de2ea001e"
-					(reference "TP8")
+					(reference "TP6")
 					(unit 1)
 				)
@@
 		(in_pos_files yes)
 		(dnp no)
-		(property "Reference" "TP10"
+		(property "Reference" "TP8"
 			(at 116.84 149.86 0)
 			(show_name no)
@@
 			(project "eumesmo-010-16ch-v1"
 				(path "/2bc5a21a-1d79-419d-a592-6852cc07b00a/7b388c9c-6faf-4681-b727-510de2ea001e"
-					(reference "TP10")
+					(reference "TP8")
 					(unit 1)
 				)
@@
 		(in_pos_files yes)
 		(dnp yes)
-		(property "Reference" "TP9"
+		(property "Reference" "TP7"
 			(at 241.3 148.59 0)
 			(show_name no)
@@
 			(project "eumesmo-010-16ch-v1"
 				(path "/2bc5a21a-1d79-419d-a592-6852cc07b00a/7b388c9c-6faf-4681-b727-510de2ea001e"
-					(reference "TP9")
+					(reference "TP7")
 					(unit 1)
 				)
@@
 		(in_pos_files yes)
 		(dnp no)
-		(property "Reference" "TP6"
+		(property "Reference" "TP4"
 			(at 224.79 116.84 0)
 			(show_name no)
@@
 			(project "eumesmo-010-16ch-v1"
 				(path "/2bc5a21a-1d79-419d-a592-6852cc07b00a/7b388c9c-6faf-4681-b727-510de2ea001e"
-					(reference "TP6")
+					(reference "TP4")
 					(unit 1)
 				)
@@
 		(in_pos_files yes)
 		(dnp no)
-		(property "Reference" "TP7"
+		(property "Reference" "TP5"
 			(at 266.7 116.84 0)
 			(show_name no)
@@
 			(project "eumesmo-010-16ch-v1"
 				(path "/2bc5a21a-1d79-419d-a592-6852cc07b00a/7b388c9c-6faf-4681-b727-510de2ea001e"
-					(reference "TP7")
+					(reference "TP5")
 					(unit 1)
 				)
