File: V1/eumesmo-010-16ch-v1-power.kicad_sch (KiCad schematic)
At the start: 55 parts, among them J5 250-202, J6 USB_C_Receptacle_USB2.0, Q1 WPM2015-3/TR, Q2 MMUN2211LT3G, U1 TX4138, U2 L78L05_SOT89, U3 B2412S-1WR3, U4 SY8089A1AAC

Commit message: Adjusted components according to availability in JLCPCB.
Parts:
- C1, C10, C11, C12, C13, C14, C15, C16, C17, C18, C2, C3, C4, C5, C6, C7, C8, C9, D1, D2, D3, D4, D5, D6, J5, J6, L1, L2, L3, Q1, Q2, R1, R10, R12, R2, R3, R4, R5, R6, R7, R8, R9, U1, U3, U4: JLCPCB BOM 1 -> (none)
- R11: value 300R -> 330R; JLCPCB BOM 1 -> (none); LCSC Part # C25102 -> C25104; Mfr PN 0402WGF3000TCE -> 0402WGF3300TCE; Vendor PN C25102 -> C25104
- TP1: value 5VSH -> TP5019; JLCPCB BOM 0 -> (none); LCSC Part # (none) -> C238131; Mfr (none) -> Keystone; Mfr PN (none) -> 5019; Vendor (none) -> JLCPCB; Vendor PN (none) -> C238131
- TP2: value 5V -> TP5019; JLCPCB BOM 0 -> (none); LCSC Part # (none) -> C238131; Mfr (none) -> Keystone; Mfr PN (none) -> 5019; Vendor (none) -> JLCPCB; Vendor PN (none) -> C238131
- TP3: value GND -> TP5019; JLCPCB BOM 0 -> (none); LCSC Part # (none) -> C238131; Mfr (none) -> Keystone; Mfr PN (none) -> 5019; Vendor (none) -> JLCPCB; Vendor PN (none) -> C238131
- TP4, TP5: JLCPCB BOM 0 -> (none); now not fitted; now left out of the parts list
- TP6, TP7: JLCPCB BOM 0 -> (none)
- TP8: value 3V3 -> TP5019; JLCPCB BOM 0 -> (none); LCSC Part # (none) -> C238131; Mfr (none) -> Keystone; Mfr PN (none) -> 5019; Vendor (none) -> JLCPCB; Vendor PN (none) -> C238131
- U2: JLCPCB BOM 1 -> (none); LCSC Part # C81154 -> C42738; Mfr PN L78L05ABD13TR -> L78L05ABUTR; Vendor PN C81154 -> C42738
Other:
- note added: "V_{F} = 2.68V @2.0mA R_{LED} = (3.3V - 2.68V) / 2.0mA R_{LED} = 0.62 / 0.002 R_{LED} = 310 ohm USE C25104 330R -> 1.88mA"
- note removed: "V_{F} = 2.68V @2.0mA R_{LED} = (3.3V - 2.68V) / 2.0mA R_{LED} = 0.62 / 0.002 R_{LED} = 310 ohm USE C25102 300R -> 2.07mA"

Commit message: RJ45 jack and terminal blocks repositioned
RJ45 jack and terminal blocks repositioned inwards the board to make space for the PCB holder. ETH tracks rerouted for better EMC.
Parts:
- TP1: now not fitted; now left out of the parts list
Changed lines of the file:
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@@
 		(body_style 1)
 		(exclude_from_sim no)
-		(in_bom yes)
-		(on_board yes)
+		(in_bom no)
+		(on_board no)
 		(in_pos_files yes)
-		(dnp no)
+		(dnp yes)
 		(property "Reference" "TP1"
 			(at 245.11 29.21 0)
@@
 		(exclude_from_sim no)
 		(in_bom no)
-		(on_board yes)
+		(on_board no)
 		(in_pos_files yes)
 		(dnp yes)
@@
 		(exclude_from_sim no)
 		(in_bom no)
-		(on_board yes)
+		(on_board no)
 		(in_pos_files yes)
 		(dnp yes)
