File: V1/eumesmo-010-16ch-v1.kicad_pcb (KiCad board)
At the start: 4 copper layers, 128 x 67.8 mm, 341 parts, among them J1 250-208, J2 250-208, J3 250-208, J4 250-208, J5 250-202, J6 250-202, J7 USB_C_Receptacle_USB2.0, J8 ETHERNET, J9 250-203, Q1 WPM2015-3/TR, Q10 MMBT2222A, Q11 MMBT2222A, Q12 MMBT2222A, Q13 MMBT2222A, Q14 MMBT2222A, Q15 MMBT2222A, Q16 MMBT2222A, Q17 MMBT2222A, Q18 MMBT2222A, Q19 MMBT2222A, Q2 MMUN2211LT3G, Q3 UMH3N, Q4 MMBT2222A, Q5 MMBT2222A, Q6 MMBT2222A, Q7 MMBT2222A, Q8 MMBT2222A, Q9 MMBT2222A, SW1 RESET, SW2 1WIRE_SEL, U1 TX4138, U10 MCP23017, U11 DS2482S-100, U12 OR-3H7-4, U13 OR-3H7-4, U14 OR-3H7-4, U15 OR-3H7-4, U2 SY8089A1AAC, U3 TPS3820-33, U4 CH340K, U5 ESP32-WROOM-32UE-N16, U6 LAN8710A, U7 TPS3823-33, U8 MCP23008, U9 MCP23008

Commit message: Development
Parts:
- removed the C15 at (192.5, 74.6)
- removed the C16 at (189.8, 74.6)
- removed the C26 at (140.3, 103.6)
- removed the C28 at (140.3, 86.3)
- removed D24, D27, D30, D33, D36, D39, D42, D45, D48, D51, D54, D57, D58, D59, D60, D61, D62, D63, D64, D65, D66, D67, D68, D69, D70, D71, D72, D73: WHITE/0603, Tales:LED_0603_1608Metric
- removed D25, D28, D31, D34, D37, D40, D43, D46, D49, D52, D55: 9V1/500mW, Tales:D_SOD-123
- removed FB1, FB10, FB11, FB12, FB13, FB14, FB15, FB16, FB2, FB3, FB4, FB5, FB6, FB7, FB8, FB9: 600R/100MHz, Tales:R_0603_1608Metric
- removed the J7 at (208.5, 71.6)
- removed J9: 250-203, Tales:TerminalBlock_Wago_250-203_1x03_P3.5mm_45Degree
- removed Q10, Q11, Q12, Q13, Q14, Q15, Q16, Q17, Q18, Q19, Q4, Q5, Q6, Q7, Q8, Q9: MMBT2222A, Tales:SOT-23-Narrow
- removed R133, R136: 10k, Tales:R_0402_1005Metric
- removed R134: 10k/100mW, Tales:R_0603_1608Metric
- removed R135: 470R, Tales:R_0402_1005Metric
- removed the R15 at (135.0, 93.6)
- removed the R16 at (135.0, 76.3)
- removed SW2: 1WIRE_SEL, Tales:SW_DIP_SPSTx02_Slide_Copal_CHS-02B_W7.62mm_P1.27mm
- removed TP9: 3V3, Tales:TestPoint_Keystone_5019_Miniature
- removed the U4 at (194.3, 70.8)
- removed the U8 at (136.3, 99.6)
- removed the U9 at (136.3, 82.3)
- added C10: 10uF/25V, Tales:C_0805_2012Metric, F.Cu at (234.5, 133.6)
- added C11: 100nF/50V, Tales:C_0402_1005Metric, F.Cu at (230.8, 133.4)
- added C19: 100nF/50V, Tales:C_0402_1005Metric, F.Cu at (249.4, 126.9)
- added C29: 100nF/50V, Tales:C_0402_1005Metric, F.Cu at (284.9, 127.0)
- added C8: 1uF/50V, Tales:C_0805_2012Metric, F.Cu at (161.3, 73.8)
- added C9: 100nF/50V, Tales:C_0402_1005Metric, F.Cu at (163.3, 73.8)
- added D11: WHITE/0603, Tales:LED_0603_1608Metric, F.Cu at (148.5, 100.8)
- added D14: WHITE/0603, Tales:LED_0603_1608Metric, F.Cu at (145.0, 105.3)
- added D17: WHITE/0603, Tales:LED_0603_1608Metric, F.Cu at (141.5, 109.8)
- added D20: WHITE/0603, Tales:LED_0603_1608Metric, F.Cu at (138.0, 114.3)
- added D23: WHITE/0603, Tales:LED_0603_1608Metric, F.Cu at (148.5, 114.3)
- added R34: 510R, Tales:R_0402_1005Metric, F.Cu at (137.8, 92.3)
- added R35: 510R, Tales:R_0402_1005Metric, F.Cu at (139.3, 92.3)
- added TP10: 3V3, Tales:TestPoint_Keystone_5019_Miniature, F.Cu at (239.6, 129.0)
- added U16: TLV274, Package_SO:TSSOP-14_4.4x5mm_P0.65mm, F.Cu at (223.1, 52.4)
- added U2: L78L05_SOT89, Package_TO_SOT_SMD:SOT-89-3, F.Cu at (157.3, 72.8)
- added U3: B2412S-1WR3, Tales:Ylptec BxxxxS-1WR3, F.Cu at (145.3, 74.8)
- added U6: CH340K, Package_SO:SSOP-10-1EP_3.9x4.9mm_P1mm_EP2.1x3.3mm, F.Cu at (249.1, 119.2)
- C31, C32: value 10uF/25V -> 100nF/50V; footprint Tales:C_0805_2012Metric -> Tales:C_0402_1005Metric
- C33, C35: value 100nF/50V -> 100nF/100V; footprint Tales:C_0402_1005Metric -> Tales:C_0805_2012Metric
- C34: value 10uF/25V -> 100nF/100V
- C36: value 470pF/50V -> 100nF/100V; footprint Tales:C_0402_1005Metric -> Tales:C_0805_2012Metric
- C37, C39, C41, C43, C49, C51, C53, C55, C57, C59, C61, C63, C65, C67: value 1nF/50V -> 100nF/100V; footprint Tales:C_0603_1608Metric -> Tales:C_0805_2012Metric
- C38, C40, C42, C44, C50, C52, C54, C56, C58, C60, C62, C64, C66, C68: value 33nF/50V -> 100nF/100V; footprint Tales:C_0603_1608Metric -> Tales:C_0805_2012Metric
- C45, C47: value 1nF/50V -> 100nF/50V; footprint Tales:C_0603_1608Metric -> Tales:C_0402_1005Metric
- C46, C48: value 33nF/50V -> 100nF/50V; footprint Tales:C_0603_1608Metric -> Tales:C_0402_1005Metric
- C7: value 100nF/50V -> 10uF/25V; footprint Tales:C_0402_1005Metric -> Tales:C_0805_2012Metric
- D10, D13, D16, D19, D22: value 9V1/500mW -> WHITE/0603; footprint Tales:D_SOD-123 -> Tales:LED_0603_1608Metric
- D8, D9: value ESD9L5.0 -> WHITE/0603; footprint Diode_SMD:D_SOD-923 -> Tales:LED_0603_1608Metric
- J6: value 250-202 -> USB_C_Receptacle_USB2.0; footprint Tales:TerminalBlock_Wago_250-202_1x02_P3.5mm_45Degree -> Tales:USB_C_Receptacle_ShouHan_TYPE-C-16PLT-H10.0
- R100, R103, R109, R112, R115, R121, R130, R91: value 10k -> 10k/125mW; footprint Tales:R_0402_1005Metric -> Tales:R_0805_2012Metric
- R101, R110, R113, R119, R122, R125, R131, R55, R61, R70, R73, R79, R82, R85, R89, R92, R95: value 10k/100mW -> 10k/125mW; footprint Tales:R_0603_1608Metric -> Tales:R_0805_2012Metric
- R102, R105, R111, R120, R123, R129, R132, R90, R93, R99: value 470R -> 10k/125mW; footprint Tales:R_0402_1005Metric -> Tales:R_0805_2012Metric
- R104, R116, R64, R76: value 10k/100mW -> 100k/125mW; footprint Tales:R_0603_1608Metric -> Tales:R_0805_2012Metric
- R106, R124, R94: value 10k -> 100k/125mW; footprint Tales:R_0402_1005Metric -> Tales:R_0805_2012Metric
- R107, R128, R58, R67, R88, R98: value 10k/100mW -> 47R/125mW; footprint Tales:R_0603_1608Metric -> Tales:R_0805_2012Metric
- R108, R117: value 470R -> 47R/125mW; footprint Tales:R_0402_1005Metric -> Tales:R_0805_2012Metric
- R114, R126, R96: value 470R -> 100k/125mW; footprint Tales:R_0402_1005Metric -> Tales:R_0805_2012Metric
- R118, R127, R97: value 10k -> 47R/125mW; footprint Tales:R_0402_1005Metric -> Tales:R_0805_2012Metric
- R36, R37, R38: value 1k -> 510R
- R39: value 1k8/125mW -> 2k2; footprint Tales:R_0805_2012Metric -> Tales:R_0402_1005Metric
- R40: value 33R -> 2k2
- R41, R44, R47, R50: value 2k2 -> 510R
- R42, R45, R48, R51: value 1k8/125mW -> 510R; footprint Tales:R_0805_2012Metric -> Tales:R_0402_1005Metric
- R43: value 10k/100mW -> 1k; footprint Tales:R_0603_1608Metric -> Tales:R_0402_1005Metric
- R46, R49, R52: value 10k/100mW -> 510R; footprint Tales:R_0603_1608Metric -> Tales:R_0402_1005Metric
- R53, R59, R62, R65, R71, R80, R83: value 2k2 -> 10k/125mW; footprint Tales:R_0402_1005Metric -> Tales:R_0805_2012Metric
- R54, R66, R84: value 1k8/125mW -> 100k/125mW
- R56, R74, R86: value 2k2 -> 100k/125mW; footprint Tales:R_0402_1005Metric -> Tales:R_0805_2012Metric
- R57, R78, R87: value 1k8/125mW -> 47R/125mW
- R60, R63, R69, R72, R75, R81: value 1k8/125mW -> 10k/125mW
- R68, R77: value 2k2 -> 47R/125mW; footprint Tales:R_0402_1005Metric -> Tales:R_0805_2012Metric
- TP16: value SDA -> SCL
- TP17: value SCL -> SDA
- U10: value MCP23017 -> ISO1540; footprint Package_SO:SSOP-28_5.3x10.2mm_P0.65mm -> Package_SO:SOIC-8_3.9x4.9mm_P1.27mm
- U11: value DS2482S-100 -> PCA9685PW; footprint Package_SO:SO-8_3.9x4.9mm_P1.27mm -> Package_SO:TSSOP-28_4.4x9.7mm_P0.65mm
- U12: value OR-3H7-4 -> MCP23017; footprint Tales:SOP-16_4.4x10.4mm_P1.27mm -> Package_SO:SSOP-28_5.3x10.2mm_P0.65mm
- U13, U14, U15: value OR-3H7-4 -> TLV274; footprint Tales:SOP-16_4.4x10.4mm_P1.27mm -> Package_SO:TSSOP-14_4.4x5mm_P0.65mm
- moved FID1 200.6 mm to (291.5, 59.4)
- moved FID3 161.8 mm to (291.5, 66.5)
- moved R70 153.0 mm to (249.9, 76.8)
- moved R69 149.5 mm to (245.5, 59.1), turned to 0 degrees
- moved R72 149.5 mm to (249.9, 79.7), turned to 0 degrees
- moved FID2 147.8 mm to (291.5, 62.9)
- moved C45 144.7 mm to (249.3, 88.1)
- moved C46 142.6 mm to (249.3, 90.0)
- moved C47 140.5 mm to (249.3, 92.0), turned to 0 degrees
- moved C54 139.8 mm to (232.4, 91.6)
- moved R82 139.0 mm to (249.9, 85.6)
- moved C53 139.0 mm to (232.4, 88.6)
- moved R79 138.9 mm to (245.5, 65.0), turned to 0 degrees
- moved C48 138.7 mm to (249.3, 94.0), turned to 0 degrees
- moved C56 137.2 mm to (232.4, 97.6), turned to 0 degrees
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- renumbered C8 to C12, C9 to C13, C10 to C14, C11 to C15, C12 to C16, C13 to C17, C14 to C18, C17 to C20, C18 to C21, C19 to C22, C20 to C23, C21 to C24, C22 to C25, C23 to C26, C24 to C27, C25 to C28, J8 to J7, R17 to R15, R18 to R16, R19 to R17, R20 to R18, R21 to R19, R22 to R20, R23 to R21, R24 to R22, R25 to R23, R26 to R24, R27 to R25, R28 to R26, R29 to R27, R30 to R28, R31 to R29, R32 to R30, R33 to R31, R34 to R32, R35 to R33, TP7 to TP6, TP6 to TP7, U2 to U4, U3 to U5, U5 to U7, U6 to U8, U7 to U9
Connections:
- C30 pad 1: +3V3 -> +5V
- C30 pad 2: GND -> GNDA
- C31 pad 1: +3V3 -> +5VA
- C31 pad 2: GND -> GNDA
- C33 pad 1: +3V3 -> /Analogs/PWM01F1
- C33 pad 2: GND -> GNDA
- C34 pad 1: +5V -> /Analogs/PWM01F2
- C34 pad 2: GND -> GNDA
- C35 pad 1: +5V -> /Analogs/PWM02F1
- C35 pad 2: GND -> GNDA
- C36 pad 1: /I2C Devices/1WIREBUS -> /Analogs/PWM02F2
- C36 pad 2: GND -> GNDA
- C37 pad 1: /IN1 -> /Analogs/PWM03F1
- C37 pad 2: GNDIO -> GNDA
- C38 pad 1: /Input 1/INFILTER -> /Analogs/PWM03F2
- C38 pad 2: GNDIO -> GNDA
- C39 pad 1: /IN2 -> /Analogs/PWM04F1
- C39 pad 2: GNDIO -> GNDA
- C40 pad 1: /Input 2/INFILTER -> /Analogs/PWM04F2
- C40 pad 2: GNDIO -> GNDA
- C41 pad 1: /IN3 -> /Analogs/PWM05F1
- C41 pad 2: GNDIO -> GNDA
- C42 pad 1: /Input 3/INFILTER -> /Analogs/PWM05F2
- C42 pad 2: GNDIO -> GNDA
- C43 pad 1: /IN4 -> /Analogs/PWM06F1
- C43 pad 2: GNDIO -> GNDA
- C44 pad 1: /Input 4/INFILTER -> /Analogs/PWM06F2
- C44 pad 2: GNDIO -> GNDA
- C45 pad 1: /IN5 -> +12VA
- C45 pad 2: GNDIO -> GNDA
- C46 pad 1: /Input 5/INFILTER -> +12VA
- C46 pad 2: GNDIO -> GNDA
- C47 pad 1: /IN6 -> +12VA
- C47 pad 2: GNDIO -> GNDA
- C48 pad 1: /Input 6/INFILTER -> +12VA
- C48 pad 2: GNDIO -> GNDA
- C49 pad 1: /IN7 -> /Analogs/PWM07F1
- C49 pad 2: GNDIO -> GNDA
- C50 pad 1: /Input 7/INFILTER -> /Analogs/PWM07F2
- C50 pad 2: GNDIO -> GNDA
- C51 pad 1: /IN8 -> /Analogs/PWM08F1
- C51 pad 2: GNDIO -> GNDA
- C52 pad 1: /Input 8/INFILTER -> /Analogs/PWM08F2
- C52 pad 2: GNDIO -> GNDA
- C53 pad 1: /IN9 -> /Analogs/PWM09F1
- C53 pad 2: GNDIO -> GNDA
- C54 pad 1: /Input 9/INFILTER -> /Analogs/PWM09F2
- C54 pad 2: GNDIO -> GNDA
- C55 pad 1: /IN10 -> /Analogs/PWM10F1
- C55 pad 2: GNDIO -> GNDA
- C56 pad 1: /Input 10/INFILTER -> /Analogs/PWM10F2
- C56 pad 2: GNDIO -> GNDA
- C57 pad 1: /IN11 -> /Analogs/PWM11F1
- C57 pad 2: GNDIO -> GNDA
- C58 pad 1: /Input 11/INFILTER -> /Analogs/PWM11F2
- C58 pad 2: GNDIO -> GNDA
- C59 pad 1: /IN12 -> /Analogs/PWM12F1
- C59 pad 2: GNDIO -> GNDA
- C6 pad 1: /Power/5VUSB -> +24V
- C60 pad 1: /Input 12/INFILTER -> /Analogs/PWM12F2
- C60 pad 2: GNDIO -> GNDA
- C61 pad 1: /IN13 -> /Analogs/PWM13F1
- C61 pad 2: GNDIO -> GNDA
- C62 pad 1: /Input 13/INFILTER -> /Analogs/PWM13F2
- C62 pad 2: GNDIO -> GNDA
- C63 pad 1: /IN14 -> /Analogs/PWM14F1
- C63 pad 2: GNDIO -> GNDA
- C64 pad 1: /Input 14/INFILTER -> /Analogs/PWM14F2
- C64 pad 2: GNDIO -> GNDA
- C65 pad 1: /IN15 -> /Analogs/PWM15F1
- C65 pad 2: GNDIO -> GNDA
- C66 pad 1: /Input 15/INFILTER -> /Analogs/PWM15F2
- C66 pad 2: GNDIO -> GNDA
- C67 pad 1: /IN16 -> /Analogs/PWM16F1
- C67 pad 2: GNDIO -> GNDA
- C68 pad 1: /Input 16/INFILTER -> /Analogs/PWM16F2
- C68 pad 2: GNDIO -> GNDA
- C7 pad 1: /Power/5VUSB -> +12VA
- C7 pad 2: GND -> GNDA
- D10 pad 1: /Input 1/INFILTER -> /I2C Devices/LDCH03A
- D10 pad 2: /Input 1/INOPTO -> +3V3
- D12 pad 1: GNDIO -> /I2C Devices/LDCH05A
- D12 pad 2: /Input 1/INLED -> +3V3
- D13 pad 1: /Input 2/INFILTER -> /I2C Devices/LDCH06A
- D13 pad 2: /Input 2/INOPTO -> +3V3
- D15 pad 1: GNDIO -> /I2C Devices/LDCH08A
- D15 pad 2: /Input 2/INLED -> +3V3
- D16 pad 1: /Input 3/INFILTER -> /I2C Devices/LDCH09A
- D16 pad 2: /Input 3/INOPTO -> +3V3
- D18 pad 1: GNDIO -> /I2C Devices/LDCH11A
- D18 pad 2: /Input 3/INLED -> +3V3
- D19 pad 1: /Input 4/INFILTER -> /I2C Devices/LDCH12A
- D19 pad 2: /Input 4/INOPTO -> +3V3
- D21 pad 1: GNDIO -> /I2C Devices/LDCH14A
- D21 pad 2: /Input 4/INLED -> +3V3
- D22 pad 1: /Input 5/INFILTER -> /I2C Devices/LDCH15A
- D22 pad 2: /Input 5/INOPTO -> +3V3
- D8 pad 1: +5V -> /I2C Devices/LDCH01A
- D8 pad 2: GND -> +3V3
- D9 pad 1: /I2C Devices/1WIREFIELD -> /I2C Devices/LDCH02A
- D9 pad 2: GND -> +3V3
- J1 pad 1: /IN1 -> /Analogs/CH01
- J1 pad 2: /IN2 -> GNDA
- J1 pad 3: /IN3 -> /Analogs/CH02
- J1 pad 4: /IN4 -> GNDA
- J1 pad 5: /IN5 -> /Analogs/CH03
- J1 pad 6: /IN6 -> GNDA
- J1 pad 7: /IN7 -> /Analogs/CH04
- J1 pad 8: /IN8 -> GNDA
- J2 pad 1: /IN9 -> /Analogs/CH05
- J2 pad 2: /IN10 -> GNDA
- J2 pad 3: /IN11 -> /Analogs/CH06
- J2 pad 4: /IN12 -> GNDA
- J2 pad 5: /IN13 -> /Analogs/CH07
- J2 pad 6: /IN14 -> GNDA
- J2 pad 7: /IN15 -> /Analogs/CH08
- J2 pad 8: /IN16 -> GNDA
- J3 pad 1: /OUT1 -> /Analogs/CH09
- J3 pad 2: /OUT2 -> GNDA
- J3 pad 3: /OUT3 -> /Analogs/CH10
- J3 pad 4: /OUT4 -> GNDA
- J3 pad 5: /OUT5 -> /Analogs/CH11
- J3 pad 6: /OUT6 -> GNDA
- J3 pad 7: /OUT7 -> /Analogs/CH12
- J3 pad 8: /OUT8 -> GNDA
- J4 pad 1: /OUT9 -> /Analogs/CH13
- J4 pad 2: /OUT10 -> GNDA
- J4 pad 3: /OUT11 -> /Analogs/CH14
- J4 pad 4: /OUT12 -> GNDA
- J4 pad 5: /OUT13 -> /Analogs/CH15
- J4 pad 6: /OUT14 -> GNDA
- J4 pad 7: /OUT15 -> /Analogs/CH16
- J4 pad 8: /OUT16 -> GNDA
- J5 pad 1: GNDIO -> /Power/+24VIN
- J5 pad 2: GNDIO -> GND
- R100 pad 1: GND -> /Analogs/CH10FB
- R100 pad 2: /OUTPUT4 -> /Analogs/CH10
- R101 pad 1: +24V -> GNDA
- R101 pad 2: /Output 5/OUTLED -> /Analogs/CH09FB
- R102 pad 1: /Output 5/OUTBASE -> GNDA
- R102 pad 2: /OUTPUT5 -> /Analogs/CH10FB
- R103 pad 1: GND -> /Analogs/PWM11
- R103 pad 2: /OUTPUT5 -> /Analogs/PWM11F1
- R104 pad 1: +24V -> /Analogs/PWM11F1
- R104 pad 2: /Output 6/OUTLED -> /Analogs/PWM11F2
- R105 pad 1: /Output 6/OUTBASE -> /Analogs/PWM12
- R105 pad 2: /OUTPUT6 -> /Analogs/PWM12F1
- R106 pad 1: GND -> /Analogs/PWM12F1
- R106 pad 2: /OUTPUT6 -> /Analogs/PWM12F2
- R107 pad 1: +24V -> /Analogs/CH11OUT
- R107 pad 2: /Output 7/OUTLED -> /Analogs/CH11
- R108 pad 1: /Output 7/OUTBASE -> /Analogs/CH12OUT
- R108 pad 2: /OUTPUT7 -> /Analogs/CH12
- R109 pad 1: GND -> /Analogs/CH11FB
- R109 pad 2: /OUTPUT7 -> /Analogs/CH11
- R110 pad 1: +24V -> /Analogs/CH12FB
- R110 pad 2: /Output 8/OUTLED -> /Analogs/CH12
- R111 pad 1: /Output 8/OUTBASE -> GNDA
- R111 pad 2: /OUTPUT8 -> /Analogs/CH11FB
- R112 pad 1: GND -> GNDA
- R112 pad 2: /OUTPUT8 -> /Analogs/CH12FB
- R113 pad 1: +24V -> /Analogs/PWM13
- R113 pad 2: /Output 9/OUTLED -> /Analogs/PWM13F1
- R114 pad 1: /Output 9/OUTBASE -> /Analogs/PWM13F1
- R114 pad 2: /OUTPUT9 -> /Analogs/PWM13F2
- R115 pad 1: GND -> /Analogs/PWM14
- R115 pad 2: /OUTPUT9 -> /Analogs/PWM14F1
- R116 pad 1: +24V -> /Analogs/PWM14F1
- R116 pad 2: /Output 10/OUTLED -> /Analogs/PWM14F2
- R117 pad 1: /Output 10/OUTBASE -> /Analogs/CH13OUT
- R117 pad 2: /OUTPUT10 -> /Analogs/CH13
- R118 pad 1: GND -> /Analogs/CH14OUT
- R118 pad 2: /OUTPUT10 -> /Analogs/CH14
- R119 pad 1: +24V -> /Analogs/CH13FB
- R119 pad 2: /Output 11/OUTLED -> /Analogs/CH13
- R120 pad 1: /Output 11/OUTBASE -> /Analogs/CH14FB
- R120 pad 2: /OUTPUT11 -> /Analogs/CH14
- R121 pad 1: GND -> GNDA
- R121 pad 2: /OUTPUT11 -> /Analogs/CH13FB
- R122 pad 1: +24V -> GNDA
- R122 pad 2: /Output 12/OUTLED -> /Analogs/CH14FB
- R123 pad 1: /Output 12/OUTBASE -> /Analogs/PWM15
- R123 pad 2: /OUTPUT12 -> /Analogs/PWM15F1
- R124 pad 1: GND -> /Analogs/PWM15F1
- R124 pad 2: /OUTPUT12 -> /Analogs/PWM15F2
- R125 pad 1: +24V -> /Analogs/PWM16
- R125 pad 2: /Output 13/OUTLED -> /Analogs/PWM16F1
- R126 pad 1: /Output 13/OUTBASE -> /Analogs/PWM16F1
- R126 pad 2: /OUTPUT13 -> /Analogs/PWM16F2
- R127 pad 1: GND -> /Analogs/CH15OUT
- R127 pad 2: /OUTPUT13 -> /Analogs/CH15
- R128 pad 1: +24V -> /Analogs/CH16OUT
- R128 pad 2: /Output 14/OUTLED -> /Analogs/CH16
- R129 pad 1: /Output 14/OUTBASE -> /Analogs/CH15FB
- R129 pad 2: /OUTPUT14 -> /Analogs/CH15
- R130 pad 1: GND -> /Analogs/CH16FB
- R130 pad 2: /OUTPUT14 -> /Analogs/CH16
- R131 pad 1: +24V -> GNDA
- R131 pad 2: /Output 15/OUTLED -> /Analogs/CH15FB
- R132 pad 1: /Output 15/OUTBASE -> GNDA
- R132 pad 2: /OUTPUT15 -> /Analogs/CH16FB
- R36 pad 1: +3V3 -> /I2C Devices/LDCH03
- R36 pad 2: /I2C Devices/MCPINN1RST -> /I2C Devices/LDCH03A
- R37 pad 1: +3V3 -> /I2C Devices/LDCH04
- R37 pad 2: /I2C Devices/MCPINN2RST -> /I2C Devices/LDCH04A
- R38 pad 1: +3V3 -> /I2C Devices/LDCH05
- R38 pad 2: /I2C Devices/MCPOUTNRST -> /I2C Devices/LDCH05A
- R39 pad 1: +3V3 -> +5VA
- R39 pad 2: /I2C Devices/1WIREBUS -> /I2C Devices/I2CSCLISO
- R40 pad 1: /I2C Devices/1WIREFIELD -> +5VA
- R40 pad 2: /I2C Devices/1WIREBUS -> /I2C Devices/I2CSDAISO
- R41 pad 1: +3V3 -> /I2C Devices/LDCH06
- R41 pad 2: /INPUT1 -> /I2C Devices/LDCH06A
- R42 pad 1: /Input 1/INFILTER -> /I2C Devices/LDCH07
- R42 pad 2: /Input 1/INPRE -> /I2C Devices/LDCH07A
- R43 pad 1: /Input 1/INPRE -> +3V3
- R43 pad 2: /Input 1/INLED -> /I2C Devices/MCPOUTNRST
- R44 pad 1: +3V3 -> /I2C Devices/LDCH08
- R44 pad 2: /INPUT2 -> /I2C Devices/LDCH08A
- R45 pad 1: /Input 2/INFILTER -> /I2C Devices/LDCH09
- R45 pad 2: /Input 2/INPRE -> /I2C Devices/LDCH09A
- R46 pad 1: /Input 2/INPRE -> /I2C Devices/LDCH10
- R46 pad 2: /Input 2/INLED -> /I2C Devices/LDCH10A
- R47 pad 1: +3V3 -> /I2C Devices/LDCH11
- R47 pad 2: /INPUT3 -> /I2C Devices/LDCH11A
- R48 pad 1: /Input 3/INFILTER -> /I2C Devices/LDCH12
- R48 pad 2: /Input 3/INPRE -> /I2C Devices/LDCH12A
- R49 pad 1: /Input 3/INPRE -> /I2C Devices/LDCH13
- R49 pad 2: /Input 3/INLED -> /I2C Devices/LDCH13A
- R50 pad 1: +3V3 -> /I2C Devices/LDCH14
- R50 pad 2: /INPUT4 -> /I2C Devices/LDCH14A
- R51 pad 1: /Input 4/INFILTER -> /I2C Devices/LDCH15
- R51 pad 2: /Input 4/INPRE -> /I2C Devices/LDCH15A
- R52 pad 1: /Input 4/INPRE -> /I2C Devices/LDCH16
- R52 pad 2: /Input 4/INLED -> /I2C Devices/LDCH16A
- R53 pad 1: +3V3 -> /Analogs/PWM01
- R53 pad 2: /INPUT5 -> /Analogs/PWM01F1
- R54 pad 1: /Input 5/INFILTER -> /Analogs/PWM01F1
- R54 pad 2: /Input 5/INPRE -> /Analogs/PWM01F2
- R55 pad 1: /Input 5/INPRE -> /Analogs/PWM02
- R55 pad 2: /Input 5/INLED -> /Analogs/PWM02F1
- R56 pad 1: +3V3 -> /Analogs/PWM02F1
- R56 pad 2: /INPUT6 -> /Analogs/PWM02F2
- R57 pad 1: /Input 6/INFILTER -> /Analogs/CH01OUT
- R57 pad 2: /Input 6/INPRE -> /Analogs/CH01
- R58 pad 1: /Input 6/INPRE -> /Analogs/CH02OUT
- R58 pad 2: /Input 6/INLED -> /Analogs/CH02
- R59 pad 1: +3V3 -> /Analogs/CH01FB
- R59 pad 2: /INPUT7 -> /Analogs/CH01
- R60 pad 1: /Input 7/INFILTER -> /Analogs/CH02FB
- R60 pad 2: /Input 7/INPRE -> /Analogs/CH02
- R61 pad 1: /Input 7/INPRE -> GNDA
- R61 pad 2: /Input 7/INLED -> /Analogs/CH01FB
- R62 pad 1: +3V3 -> GNDA
- R62 pad 2: /INPUT8 -> /Analogs/CH02FB
- R63 pad 1: /Input 8/INFILTER -> /Analogs/PWM03
- R63 pad 2: /Input 8/INPRE -> /Analogs/PWM03F1
- R64 pad 1: /Input 8/INPRE -> /Analogs/PWM03F1
- R64 pad 2: /Input 8/INLED -> /Analogs/PWM03F2
- R65 pad 1: +3V3 -> /Analogs/PWM04
- R65 pad 2: /INPUT9 -> /Analogs/PWM04F1
- R66 pad 1: /Input 9/INFILTER -> /Analogs/PWM04F1
- R66 pad 2: /Input 9/INPRE -> /Analogs/PWM04F2
- R67 pad 1: /Input 9/INPRE -> /Analogs/CH03OUT
- R67 pad 2: /Input 9/INLED -> /Analogs/CH03
- R68 pad 1: +3V3 -> /Analogs/CH04OUT
- R68 pad 2: /INPUT10 -> /Analogs/CH04
- R69 pad 1: /Input 10/INFILTER -> /Analogs/CH03FB
- R69 pad 2: /Input 10/INPRE -> /Analogs/CH03
- R70 pad 1: /Input 10/INPRE -> /Analogs/CH04FB
- R70 pad 2: /Input 10/INLED -> /Analogs/CH04
- R71 pad 1: +3V3 -> GNDA
- R71 pad 2: /INPUT11 -> /Analogs/CH03FB
- R72 pad 1: /Input 11/INFILTER -> GNDA
- R72 pad 2: /Input 11/INPRE -> /Analogs/CH04FB
- R73 pad 1: /Input 11/INPRE -> /Analogs/PWM05
- R73 pad 2: /Input 11/INLED -> /Analogs/PWM05F1
- R74 pad 1: +3V3 -> /Analogs/PWM05F1
- R74 pad 2: /INPUT12 -> /Analogs/PWM05F2
- R75 pad 1: /Input 12/INFILTER -> /Analogs/PWM06
- R75 pad 2: /Input 12/INPRE -> /Analogs/PWM06F1
- R76 pad 1: /Input 12/INPRE -> /Analogs/PWM06F1
- R76 pad 2: /Input 12/INLED -> /Analogs/PWM06F2
- R77 pad 1: +3V3 -> /Analogs/CH05OUT
- R77 pad 2: /INPUT13 -> /Analogs/CH05
- R78 pad 1: /Input 13/INFILTER -> /Analogs/CH06OUT
- R78 pad 2: /Input 13/INPRE -> /Analogs/CH06
- R79 pad 1: /Input 13/INPRE -> /Analogs/CH05FB
- R79 pad 2: /Input 13/INLED -> /Analogs/CH05
- R80 pad 1: +3V3 -> /Analogs/CH06FB
- R80 pad 2: /INPUT14 -> /Analogs/CH06
- R81 pad 1: /Input 14/INFILTER -> GNDA
- R81 pad 2: /Input 14/INPRE -> /Analogs/CH05FB
- R82 pad 1: /Input 14/INPRE -> GNDA
- R82 pad 2: /Input 14/INLED -> /Analogs/CH06FB
- R83 pad 1: +3V3 -> /Analogs/PWM07
- R83 pad 2: /INPUT15 -> /Analogs/PWM07F1
- R84 pad 1: /Input 15/INFILTER -> /Analogs/PWM07F1
- R84 pad 2: /Input 15/INPRE -> /Analogs/PWM07F2
- R85 pad 1: /Input 15/INPRE -> /Analogs/PWM08
- R85 pad 2: /Input 15/INLED -> /Analogs/PWM08F1
- R86 pad 1: +3V3 -> /Analogs/PWM08F1
- R86 pad 2: /INPUT16 -> /Analogs/PWM08F2
- R87 pad 1: /Input 16/INFILTER -> /Analogs/CH07OUT
- R87 pad 2: /Input 16/INPRE -> /Analogs/CH07
- R88 pad 1: /Input 16/INPRE -> /Analogs/CH08OUT
- R88 pad 2: /Input 16/INLED -> /Analogs/CH08
- R89 pad 1: +24V -> /Analogs/CH07FB
- R89 pad 2: /Output 1/OUTLED -> /Analogs/CH07
- R90 pad 1: /Output 1/OUTBASE -> /Analogs/CH08FB
- R90 pad 2: /OUTPUT1 -> /Analogs/CH08
- R91 pad 1: GND -> GNDA
- R91 pad 2: /OUTPUT1 -> /Analogs/CH07FB
- R92 pad 1: +24V -> GNDA
- R92 pad 2: /Output 2/OUTLED -> /Analogs/CH08FB
- R93 pad 1: /Output 2/OUTBASE -> /Analogs/PWM09
- R93 pad 2: /OUTPUT2 -> /Analogs/PWM09F1
- R94 pad 1: GND -> /Analogs/PWM09F1
- R94 pad 2: /OUTPUT2 -> /Analogs/PWM09F2
- R95 pad 1: +24V -> /Analogs/PWM10
- R95 pad 2: /Output 3/OUTLED -> /Analogs/PWM10F1
- R96 pad 1: /Output 3/OUTBASE -> /Analogs/PWM10F1
- R96 pad 2: /OUTPUT3 -> /Analogs/PWM10F2
- R97 pad 1: GND -> /Analogs/CH09OUT
- R97 pad 2: /OUTPUT3 -> /Analogs/CH09
- R98 pad 1: +24V -> /Analogs/CH10OUT
- R98 pad 2: /Output 4/OUTLED -> /Analogs/CH10
- R99 pad 1: /Output 4/OUTBASE -> /Analogs/CH09FB
- R99 pad 2: /OUTPUT4 -> /Analogs/CH09
- TP16 pad 1: /I2C Devices/I2CSDA -> /I2C Devices/I2CSCL
- TP17 pad 1: /I2C Devices/I2CSCL -> /I2C Devices/I2CSDA
- U10 pad 1: /OUTPUT9 -> +5V
- U10 pad 2: /OUTPUT10 -> /I2C Devices/I2CSDA
- U10 pad 3: /OUTPUT11 -> /I2C Devices/I2CSCL
- U10 pad 4: /OUTPUT12 -> GND
- U10 pad 5: /OUTPUT13 -> GNDA
- U10 pad 6: /OUTPUT14 -> /I2C Devices/I2CSCLISO
- U10 pad 7: /OUTPUT15 -> /I2C Devices/I2CSDAISO
- U10 pad 8: /OUTPUT16 -> +5VA
- U11 pad 1: +3V3 -> GNDA
- U11 pad 2: /I2C Devices/1WIREMASTER -> GNDA
- U11 pad 3: GND -> GNDA
- U11 pad 4: /I2C Devices/I2CSCL -> GNDA
- U11 pad 5: /I2C Devices/I2CSDA -> GNDA
- U11 pad 6: unconnected-(U11-PCTLZ-Pad6) -> /Analogs/PWM01
- U11 pad 7: GND -> /Analogs/PWM02
- U11 pad 8: GND -> /Analogs/PWM03
- U12 pad 1: /Input 4/INOPTO -> /I2C Devices/LDCH09
- U12 pad 10: /INPUT1 -> GND
- U12 pad 11: GND -> unconnected-(U12-NC-Pad11)
- U12 pad 12: /INPUT2 -> /I2C Devices/I2CSCL
- U12 pad 13: GND -> /I2C Devices/I2CSDA
- U12 pad 14: /INPUT3 -> unconnected-(U12-NC-Pad14)
- U12 pad 16: /INPUT4 -> GND
- U12 pad 2: GNDIO -> /I2C Devices/LDCH10
- U12 pad 3: /Input 3/INOPTO -> /I2C Devices/LDCH11
- U12 pad 4: GNDIO -> /I2C Devices/LDCH12
- U12 pad 5: /Input 2/INOPTO -> /I2C Devices/LDCH13
- U12 pad 6: GNDIO -> /I2C Devices/LDCH14
- U12 pad 7: /Input 1/INOPTO -> /I2C Devices/LDCH15
- U12 pad 8: GNDIO -> /I2C Devices/LDCH16
- U12 pad 9: GND -> +3V3
- U13 pad 1: /Input 8/INOPTO -> /Analogs/CH01OUT
- U13 pad 10: /INPUT5 -> /Analogs/PWM03F2
- U13 pad 11: GND -> GNDA
- U13 pad 12: /INPUT6 -> /Analogs/PWM04F2
- U13 pad 13: GND -> /Analogs/CH04FB
- U13 pad 14: /INPUT7 -> /Analogs/CH04OUT
- U13 pad 2: GNDIO -> /Analogs/CH01FB
- U13 pad 3: /Input 7/INOPTO -> /Analogs/PWM01F2
- U13 pad 4: GNDIO -> +12VA
- U13 pad 5: /Input 6/INOPTO -> /Analogs/PWM02F2
- U13 pad 6: GNDIO -> /Analogs/CH02FB
- U13 pad 7: /Input 5/INOPTO -> /Analogs/CH02OUT
- U13 pad 8: GNDIO -> /Analogs/CH03OUT
- U13 pad 9: GND -> /Analogs/CH03FB
- U14 pad 1: /Input 12/INOPTO -> /Analogs/CH05OUT
- U14 pad 10: /INPUT9 -> /Analogs/PWM07F2
- U14 pad 11: GND -> GNDA
- U14 pad 12: /INPUT10 -> /Analogs/PWM08F2
- U14 pad 13: GND -> /Analogs/CH08FB
- U14 pad 14: /INPUT11 -> /Analogs/CH08OUT
- U14 pad 2: GNDIO -> /Analogs/CH05FB
- U14 pad 3: /Input 11/INOPTO -> /Analogs/PWM05F2
- U14 pad 4: GNDIO -> +12VA
- U14 pad 5: /Input 10/INOPTO -> /Analogs/PWM06F2
- U14 pad 6: GNDIO -> /Analogs/CH06FB
- U14 pad 7: /Input 9/INOPTO -> /Analogs/CH06OUT
- U14 pad 8: GNDIO -> /Analogs/CH07OUT
- U14 pad 9: GND -> /Analogs/CH07FB
- U15 pad 1: /Input 16/INOPTO -> /Analogs/CH09OUT
- U15 pad 10: /INPUT13 -> /Analogs/PWM11F2
- U15 pad 11: GND -> GNDA
- U15 pad 12: /INPUT14 -> /Analogs/PWM12F2
- U15 pad 13: GND -> /Analogs/CH12FB
- U15 pad 14: /INPUT15 -> /Analogs/CH12OUT
- U15 pad 2: GNDIO -> /Analogs/CH09FB
- U15 pad 3: /Input 15/INOPTO -> /Analogs/PWM09F2
- U15 pad 4: GNDIO -> +12VA
- U15 pad 5: /Input 14/INOPTO -> /Analogs/PWM10F2
- U15 pad 6: GNDIO -> /Analogs/CH10FB
- U15 pad 7: /Input 13/INOPTO -> /Analogs/CH10OUT
- U15 pad 8: GNDIO -> /Analogs/CH11OUT
- U15 pad 9: GND -> /Analogs/CH11FB
- U7 pad 13: /I2C Devices/MCPIN2INT -> unconnected-(U7-IO14-Pad13)
- U7 pad 16: /I2C Devices/MCPIN1INT -> unconnected-(U7-IO13-Pad16)
- U7 pad 27: /I2C Devices/1WIREGPIO -> unconnected-(U7-IO16-Pad27)
Routing:
- net +3V3: track 141.5 -> 8.58 mm, vias 34 -> 15
- net /I2C Devices/I2CSCL: track 102.9 -> 2.05 mm, vias 4 -> 0
- net /I2C Devices/I2CSDA: track 100.9 -> 2.04 mm, vias 4 -> 0
- net GND: track 132.7 -> 34.6 mm, vias 140 -> 63
- net /Power/5VUSB: track 83.1 -> 0.00 mm, vias 6 -> 0
- net GNDIO: track 64.2 -> 0.00 mm, vias 40 -> 0
- net /I2C Devices/MCPIN2INT: track 46.8 -> 0.00 mm, vias 4 -> 0
- net /OUTPUT16: track 45.8 -> 0.00 mm, vias 2 -> 0
- net /I2C Devices/MCPIN1INT: track 43.5 -> 0.00 mm, vias 2 -> 0
- net /OUTPUT15: track 40.7 -> 0.00 mm, vias 2 -> 0
- net /Input 9/INOPTO: track 39.4 -> 0.00 mm, vias 2 -> 0
- net /OUTPUT14: track 37.4 -> 0.00 mm, vias 2 -> 0
- net /MCU/MRESET: track 39.6 -> 3.40 mm
- net /OUTPUT13: track 35.5 -> 0.00 mm, vias 2 -> 0
- net /Input 10/INOPTO: track 34.3 -> 0.00 mm, vias 2 -> 0
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- removed copper zone on In2.Cu, net +24V
- removed copper zone on In1.Cu, net GNDIO
Other:
- board text added: "eumesmo-010-16ch"
- board text removed: "+5V"
- board text removed: "0V INPUTS"
- board text removed: "1-WIRE INTERFACE"
- board text removed: "1W"
- board text removed: "DS2482"
- board text removed: "GPIO16"
- board text removed: "I1"
- board text removed: "I10"
- board text removed: "I11"
- board text removed: "I12"
- board text removed: "I13"
- board text removed: "I14"
- board text removed: "I15"
- board text removed: "I16"
- board text removed: "I2"
- board text removed: "I3"
- board text removed: "I4"
- board text removed: "I5"
- board text removed: "I6"
- board text removed: "I7"
- board text removed: "I8"
- board text removed: "I9"
- board text removed: "O1"
- board text removed: "O10"
- board text removed: "O11"
- board text removed: "O12"
- board text removed: "O13"
- board text removed: "O14"
- board text removed: "O15"
- board text removed: "O16"
- board text removed: "O2"
- board text removed: "O3"
- board text removed: "O4"
- board text removed: "O5"
- board text removed: "O6"
- board text removed: "O7"
- board text removed: "O8"
- board text removed: "O9"
- board text removed: "eumesmo-io-24v16ch"

Commit message: Development
Parts:
- added D24: WHITE/0603, Tales:LED_0603_1608Metric, F.Cu at (135.8, 57.3)
- added R133: 300R, Tales:R_0402_1005Metric, F.Cu at (138.8, 57.3)
- added REF**: Icon_Power_Plug, Tales:Icon_Power_Plug, F.Cu at (129.8, 53.3)
- added REF**: Icon_Heart_Flash, Tales:Icon_Heart_Flash, F.Cu at (129.8, 57.3)
- R11: value 1k -> 300R
- R34, R35, R36, R37, R38, R41, R42, R44, R45, R46, R47, R48, R49, R50, R51, R52: value 510R -> 300R
- moved TP12 156.1 mm to (97.8, 79.6)
- moved TP11 155.8 mm to (97.8, 77.1)
- moved Q3 152.2 mm to (103.3, 83.6)
- moved U6 151.2 mm to (103.3, 79.1)
- moved C10 150.1 mm to (93.8, 81.3), turned to 180 degrees
- moved C19 149.7 mm to (106.3, 83.1)
- moved C11 146.0 mm to (93.8, 83.1), turned to 180 degrees
- moved J6 141.9 mm to (96.3, 71.1)
- moved D5 141.2 mm to (93.8, 78.1)
- moved R6 140.3 mm to (102.3, 69.1), turned to -90 degrees
- moved R7 139.4 mm to (102.3, 73.1), turned to 90 degrees
- moved R69 83.7 mm to (182.1, 113.6)
- moved R71 83.7 mm to (182.1, 116.6)
- moved D6 54.8 mm to (135.8, 55.6), turned to 0 degrees
- moved R11 53.8 mm to (138.8, 55.6), turned to 180 degrees
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Connections:
- net /Power/5VLED renamed /Power/3V3LED
- D5 pad 1: /Power/USBCD- -> /Power/USBCD+
- D5 pad 3: /Power/USBCD+ -> /Power/USBCD-
- D5 pad 4: /MCU/USBD+ -> /MCU/USBD-
- D5 pad 6: /MCU/USBD- -> /MCU/USBD+
- R11 pad 1: +5V -> +3V3
- U7 pad 24: unconnected-(U7-IO2-Pad24) -> /MCU/CPUOK
Routing:
- net /MCU/ESPPROG: track 25.0 -> 2.83 mm, vias 2 -> 0
- net +3V3: track 8.58 -> 0.74 mm, vias 15 -> 12
- net /Power/3V3LED: track 1.70 -> 0.00 mm
Other:
- board text added: "V1.0 2026-06-21"
- board text removed: "5V"
- board text removed: "V6.2 2026-06-17"
