File: V1/eumesmo-010-16ch-v1.kicad_pcb (KiCad board)
At the start: 4 copper layers, 128 x 67.8 mm, 275 parts, among them J1 250-208, J2 250-208, J3 250-208, J4 250-208, J5 250-202, J6 USB_C_Receptacle_USB2.0, J7 ETHERNET, Q1 WPM2015-3/TR, Q2 MMUN2211LT3G, Q3 UMH3N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

Commit message: Development
Parts:
- removed TP10: 3V3, Tales:TestPoint_Keystone_5019_Miniature
- removed TP11: D+, TestPoint:TestPoint_Pad_D1.5mm
- removed TP12: D-, TestPoint:TestPoint_Pad_D1.5mm
- removed TP16: SCL, TestPoint:TestPoint_Pad_D1.5mm
- removed TP17: SDA, TestPoint:TestPoint_Pad_D1.5mm
- removed TP3, TP5: GND, Tales:TestPoint_Keystone_5019_Miniature
- moved C30 143.3 mm to (162.6, 54.4)
- moved C29 143.3 mm to (162.6, 52.5)
- moved C31 143.3 mm to (162.6, 56.4)
- moved R39 114.0 mm to (181.3, 42.7)
- moved R40 114.0 mm to (181.3, 44.7)
- moved U10 114.0 mm to (184.0, 56.2)
- moved R100 94.4 mm to (163.5, 90.8), turned to 180 degrees
- moved R102 90.3 mm to (167.0, 90.8), turned to 180 degrees
- moved R112 83.9 mm to (170.5, 78.3)
- moved R72 83.6 mm to (170.5, 105.8)
- moved C45 82.9 mm to (168.8, 108.1), turned to 90 degrees
- moved R99 82.0 mm to (163.5, 78.3), turned to 180 degrees
- moved R70 81.3 mm to (174.0, 105.8)
- moved C47 81.3 mm to (168.8, 80.6), turned to 90 degrees
- moved R110 80.7 mm to (174.0, 78.3)
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Routing:
- net GNDA: track 3.79 -> 47.2 mm, vias 4 -> 52
- net +12VA: track 0.00 -> 23.2 mm
- net /Analogs/CH04FB: track 0.00 -> 17.5 mm
- net /Analogs/CH14FB: track 0.00 -> 8.77 mm
- net /Analogs/CH10FB: track 0.00 -> 8.77 mm
- net /Analogs/CH06FB: track 0.00 -> 8.77 mm
- net /Analogs/CH13FB: track 0.00 -> 8.77 mm
- net /Analogs/CH09FB: track 0.00 -> 8.77 mm
- net /Analogs/CH05FB: track 0.00 -> 8.77 mm
- net /Analogs/CH15FB: track 0.00 -> 8.77 mm
- net /Analogs/CH07FB: track 0.00 -> 8.77 mm
- net /Analogs/CH03FB: track 0.00 -> 8.77 mm
- net /Analogs/CH11FB: track 0.00 -> 8.77 mm
- net /Analogs/CH16FB: track 0.00 -> 8.77 mm
- net /Analogs/CH12FB: track 0.00 -> 8.77 mm
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- added copper zone on In1.Cu, net GNDA

Commit message: Development
Parts:
- moved R39 45.2 mm to (152.5, 77.6), turned to 180 degrees
- moved R40 42.5 mm to (152.5, 76.1), turned to 180 degrees
- moved U10 41.7 mm to (147.8, 76.8)
- moved C29 30.5 mm to (188.0, 69.3)
- moved C30 28.3 mm to (143.0, 74.8), turned to 180 degrees
- moved C31 21.0 mm to (152.5, 74.8)
- moved U11 12.9 mm to (184.3, 74.8), turned to 0 degrees
- moved C8 8.43 mm to (169.5, 73.3), turned to 0 degrees
- moved U2 7.32 mm to (164.5, 71.6), turned to 180 degrees
- moved C9 5.76 mm to (169.0, 71.8), turned to 0 degrees
- turned R90 to 0 degrees
Routing:
- net /Analogs/CH08: track 0.00 -> 20.7 mm, vias 0 -> 1
- net /Analogs/CH16: track 3.82 -> 20.7 mm, vias 0 -> 1
- net /Analogs/CH12: track 3.82 -> 20.7 mm, vias 0 -> 1
- net /Analogs/CH09: track 3.82 -> 20.4 mm, vias 0 -> 1
- net /Analogs/CH01: track 3.82 -> 20.4 mm, vias 0 -> 1
- net /Analogs/CH13: track 3.82 -> 20.4 mm, vias 0 -> 1
- net /Analogs/CH05: track 3.82 -> 20.4 mm, vias 0 -> 1
- net GNDA: track 47.2 -> 60.2 mm, vias 52 -> 60
- net /Analogs/CH04: track 7.64 -> 20.7 mm, vias 0 -> 1
- net /Analogs/CH04FB: track 17.5 -> 8.77 mm
- net /Analogs/CH08FB: track 0.00 -> 8.77 mm
- net /Analogs/CH14: track 3.82 -> 8.78 mm
- net /Analogs/CH10: track 3.82 -> 8.78 mm
- net /Analogs/CH06: track 3.82 -> 8.78 mm
- net /Analogs/CH02: track 3.82 -> 8.78 mm
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
Commit message: Development
Parts:
- added C69: 100pF/50V, Tales:C_0805_2012Metric, F.Cu at (163.5, 105.8)
- added C70: 100pF/50V, Tales:C_0805_2012Metric, F.Cu at (163.5, 118.3)
- added C71: 100pF/50V, Tales:C_0805_2012Metric, F.Cu at (174.0, 118.3)
- added C72: 100pF/50V, Tales:C_0805_2012Metric, F.Cu at (174.0, 105.8)
- added C73: 100pF/50V, Tales:C_0805_2012Metric, F.Cu at (194.5, 105.8)
- added C74: 100pF/50V, Tales:C_0805_2012Metric, F.Cu at (194.5, 118.3)
- added C75: 100pF/50V, Tales:C_0805_2012Metric, F.Cu at (205.0, 118.3)
- added C76: 100pF/50V, Tales:C_0805_2012Metric, F.Cu at (205.0, 105.8)
- added C77: 100pF/50V, Tales:C_0805_2012Metric, F.Cu at (163.5, 68.6)
- added C78: 100pF/50V, Tales:C_0805_2012Metric, F.Cu at (163.5, 81.1)
- added C79: 100pF/50V, Tales:C_0805_2012Metric, F.Cu at (174.0, 81.1)
- added C80: 100pF/50V, Tales:C_0805_2012Metric, F.Cu at (174.0, 68.6)
- added C81: 100pF/50V, Tales:C_0805_2012Metric, F.Cu at (194.5, 68.6)
- added C82: 100pF/50V, Tales:C_0805_2012Metric, F.Cu at (194.5, 81.1)
- added C83: 100pF/50V, Tales:C_0805_2012Metric, F.Cu at (205.0, 81.1)
- added C84: 100pF/50V, Tales:C_0805_2012Metric, F.Cu at (205.0, 68.6)
- added TP10: 3V3, Tales:TestPoint_Keystone_5019_Miniature, F.Cu at (165.9, 52.5)
- added TP11: D+, TestPoint:TestPoint_Pad_D1.5mm, F.Cu at (172.5, 53.5)
- added TP12: D-, TestPoint:TestPoint_Pad_D1.5mm, F.Cu at (172.5, 57.0)
- added TP16: SCL, TestPoint:TestPoint_Pad_D1.5mm, F.Cu at (172.5, 44.4)
- added TP17: SDA, TestPoint:TestPoint_Pad_D1.5mm, F.Cu at (172.5, 47.9)
- added TP3: GND, Tales:TestPoint_Keystone_5019_Miniature, F.Cu at (165.9, 44.6)
- added TP5: GND, Tales:TestPoint_Keystone_5019_Miniature, F.Cu at (165.9, 48.5)
- R100, R109, R110, R119, R120, R129, R130, R59, R60, R69, R70, R79, R80, R89, R90, R99: value 10k/125mW -> 11k/125mW
- R104, R106, R114, R116, R124, R126, R54, R56, R64, R66, R74, R76, R84, R86, R94, R96: value 100k/125mW -> 10k/125mW
- moved C29 29.3 mm to (178.8, 97.1), turned to 90 degrees
- moved U11 26.0 mm to (184.3, 100.8), turned to 90 degrees
- moved R108 13.3 mm to (177.5, 68.6)
- moved R117 13.3 mm to (191.0, 68.6)
- moved R128 13.3 mm to (208.5, 68.6)
- moved R97 13.3 mm to (160.0, 68.6)
- moved R100 12.2 mm to (165.8, 78.8)
- moved R109 12.2 mm to (171.8, 78.8)
- moved R120 12.2 mm to (196.8, 78.8)
- moved R129 12.2 mm to (202.8, 78.8)
- moved C47 9.75 mm to (168.8, 70.8)
- moved C48 9.75 mm to (199.8, 70.8)
- moved C53 9.75 mm to (158.8, 71.8)
- moved C54 9.75 mm to (162.3, 71.8)
- moved C55 9.75 mm to (158.8, 77.8)
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Connections:
- R100 pad 2: /Analogs/CH10 -> /Analogs/CH10OUT
- R109 pad 2: /Analogs/CH11 -> /Analogs/CH11OUT
- R110 pad 2: /Analogs/CH12 -> /Analogs/CH12OUT
- R119 pad 2: /Analogs/CH13 -> /Analogs/CH13OUT
- R120 pad 2: /Analogs/CH14 -> /Analogs/CH14OUT
- R129 pad 2: /Analogs/CH15 -> /Analogs/CH15OUT
- R130 pad 2: /Analogs/CH16 -> /Analogs/CH16OUT
- R59 pad 2: /Analogs/CH01 -> /Analogs/CH01OUT
- R60 pad 2: /Analogs/CH02 -> /Analogs/CH02OUT
- R69 pad 2: /Analogs/CH03 -> /Analogs/CH03OUT
- R70 pad 2: /Analogs/CH04 -> /Analogs/CH04OUT
- R79 pad 2: /Analogs/CH05 -> /Analogs/CH05OUT
- R80 pad 2: /Analogs/CH06 -> /Analogs/CH06OUT
- R89 pad 2: /Analogs/CH07 -> /Analogs/CH07OUT
- R90 pad 2: /Analogs/CH08 -> /Analogs/CH08OUT
- R99 pad 2: /Analogs/CH09 -> /Analogs/CH09OUT
Routing:
- net /Analogs/CH15OUT: track 2.37 -> 7.96 mm
- net /Analogs/CH11OUT: track 2.37 -> 7.96 mm
- net /Analogs/CH07OUT: track 2.37 -> 7.96 mm
- net /Analogs/CH03OUT: track 2.37 -> 7.96 mm
- net /Analogs/CH16OUT: track 2.37 -> 7.96 mm
- net /Analogs/CH04OUT: track 2.37 -> 7.96 mm
- net /Analogs/CH12OUT: track 2.37 -> 7.96 mm
- net /Analogs/CH08OUT: track 2.37 -> 7.96 mm
- net /Analogs/CH14OUT: track 2.37 -> 7.96 mm
- net /Analogs/CH10OUT: track 2.37 -> 7.96 mm
- net /Analogs/CH06OUT: track 2.37 -> 7.96 mm
- net /Analogs/CH02OUT: track 2.37 -> 7.96 mm
- net /Analogs/CH09OUT: track 2.37 -> 7.96 mm
- net /Analogs/CH05OUT: track 2.37 -> 7.96 mm
- net /Analogs/CH01OUT: track 2.37 -> 7.96 mm
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
Commit message: Development
Parts:
- removed TP10: 3V3, Tales:TestPoint_Keystone_5019_Miniature
- removed TP11: D+, TestPoint:TestPoint_Pad_D1.5mm
- removed TP12: D-, TestPoint:TestPoint_Pad_D1.5mm
- removed TP16: SCL, TestPoint:TestPoint_Pad_D1.5mm
- removed TP17: SDA, TestPoint:TestPoint_Pad_D1.5mm
- removed TP2: 5V, Tales:TestPoint_Keystone_5019_Miniature
- removed TP3, TP5: GND, Tales:TestPoint_Keystone_5019_Miniature
- removed TP7: 3V3A, TestPoint:TestPoint_Pad_D1.5mm
- moved G*** 70.5 mm to (167.0, 100.6)
- moved C29 1.35 mm to (178.3, 98.3), turned to -90 degrees
Routing:
- net /Analogs/PWM16: track 0.00 -> 57.9 mm
- net /Analogs/PWM09: track 0.00 -> 57.3 mm, vias 0 -> 2
- net /Analogs/PWM10: track 0.00 -> 53.7 mm, vias 0 -> 2
- net /Analogs/PWM15: track 0.00 -> 52.9 mm
- net /Analogs/PWM02: track 0.00 -> 43.4 mm
- net /Analogs/PWM07: track 0.00 -> 41.5 mm
- net /Analogs/PWM01: track 0.00 -> 38.3 mm
- net /Analogs/PWM08: track 0.00 -> 36.7 mm
- net /Analogs/PWM12: track 0.00 -> 32.6 mm, vias 0 -> 2
- net /Analogs/PWM11: track 0.00 -> 31.5 mm, vias 0 -> 2
- net /Analogs/PWM13: track 0.00 -> 28.5 mm, vias 0 -> 2
- net /Analogs/PWM14: track 0.00 -> 24.6 mm
- net /Analogs/PWM03: track 0.00 -> 13.5 mm
- net /Analogs/PWM04: track 0.00 -> 11.9 mm, vias 0 -> 2
- net /Analogs/PWM06: track 0.00 -> 10.8 mm
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Other:
- board text added: "+ CH01 -"
- board text added: "+ CH02 -"
- board text added: "+ CH03 -"
- board text added: "+ CH04 -"
- board text added: "+ CH05 -"
- board text added: "+ CH06 -"
- board text added: "+ CH07 -"
- board text added: "+ CH08 -"
- board text added: "+ CH09 -"
- board text added: "+ CH10 -"
- board text added: "+ CH11 -"
- board text added: "+ CH12 -"
- board text added: "+ CH13 -"
- board text added: "+ CH14 -"
- board text added: "+ CH15 -"
- board text added: "+ CH16 -"

Commit message: Development
Parts:
- removed TP1: 5VSH, Tales:TestPoint_Keystone_5019_Miniature
- removed TP15: CLK, TestPoint:TestPoint_Pad_D1.5mm
- removed TP4: GND, Tales:TestPoint_Keystone_5019_Miniature
- removed TP6: 3V3LAN, TestPoint:TestPoint_Pad_D1.5mm
- moved D20 18.3 mm to (137.8, 96.1), turned to 0 degrees
- moved D21 18.3 mm to (141.3, 96.1), turned to 0 degrees
- moved D22 18.3 mm to (144.8, 96.1), turned to 0 degrees
- moved D23 18.3 mm to (148.3, 96.1), turned to 0 degrees
- moved R37 17.2 mm to (148.0, 108.6), turned to 180 degrees
- moved R36 16.7 mm to (144.5, 108.6), turned to 180 degrees
- moved R35 16.3 mm to (141.0, 108.6), turned to 180 degrees
- moved R34 16.3 mm to (137.5, 108.6), turned to 180 degrees
- moved R38 13.1 mm to (137.5, 103.8), turned to 180 degrees
- moved R43 12.8 mm to (149.8, 88.3)
- moved R41 12.3 mm to (141.0, 103.8), turned to 180 degrees
- moved R42 11.7 mm to (144.5, 103.8), turned to 180 degrees
- moved R44 11.5 mm to (148.0, 103.8), turned to 180 degrees
- moved D10 9.50 mm to (144.8, 110.3), turned to 0 degrees
- moved D11 9.50 mm to (148.3, 110.3), turned to 0 degrees
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Routing:
- net /I2C Devices/LDCH05: track 0.00 -> 33.3 mm
- net /I2C Devices/LDCH06: track 0.00 -> 30.7 mm
- net /I2C Devices/I2CSCLISO: track 0.00 -> 30.3 mm
- net /I2C Devices/LDCH12: track 0.00 -> 29.3 mm
- net /I2C Devices/LDCH07: track 0.00 -> 29.0 mm
- net /I2C Devices/LDCH01: track 0.00 -> 29.0 mm, vias 0 -> 2
- net /I2C Devices/LDCH02: track 0.00 -> 28.8 mm, vias 0 -> 2
- net /I2C Devices/LDCH03: track 0.00 -> 28.6 mm, vias 0 -> 2
- net /I2C Devices/LDCH04: track 0.00 -> 28.6 mm, vias 0 -> 2
- net /I2C Devices/I2CSDAISO: track 0.00 -> 28.4 mm
- net /I2C Devices/LDCH11: track 0.00 -> 27.4 mm
- net /I2C Devices/LDCH08: track 0.00 -> 27.2 mm
- net /I2C Devices/LDCH10: track 0.00 -> 25.5 mm
- net /I2C Devices/LDCH09: track 0.00 -> 23.5 mm
- net /I2C Devices/LDCH16: track 0.00 -> 17.1 mm
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Other:
- board text added: "CH01"
- board text added: "CH02"
- board text added: "CH03"
- board text added: "CH04"
- board text added: "CH05"
- board text added: "CH06"
- board text added: "CH07"
- board text added: "CH08"
- board text added: "CH09"
- board text added: "CH10"
- board text added: "CH11"
- board text added: "CH12"
- board text added: "CH13"
- board text added: "CH14"
- board text added: "CH15"
- board text added: "CH16"
