File: V1/eumesmo-010-16ch-v1.kicad_pcb (KiCad board)
At the start: 4 copper layers, 128 x 67.8 mm, 284 parts, among them J1 250-208, J2 250-208, J3 250-208, J4 250-208, J5 250-202, J6 USB_C_Receptacle_USB2.0, J7 ETHERNET, Q1 WPM2015-3/TR, Q2 MMUN2211LT3G, Q3 UMH3N, SW1 RESET, U1 TX4138, U10 ISO1540, U11 PCA9685PW, U12 MCP23017, U13 TLV274, U14 TLV274, U15 TLV274, U16 TLV274, U2 L78L05_SOT89, U3 B2412S-1WR3, U4 SY8089A1AAC, U5 TPS3820-33, U6 CH340K, U7 ESP32-WROOM-32UE-N16, U8 LAN8710A, U9 TPS3823-33

Commit message: Added CPU health LED
Other:
- board text added: "V1.0 2026-07-02"
- board text removed: "V1.0 2026-06-23"
Changed lines of the file:
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@@
 		(layer "Edge.Cuts")
 	)
-	(gr_text "V1.0 2026-06-23"
+	(gr_text "V1.0 2026-07-02"
 		(at 109.52 133.08 0)
 		(layer "F.SilkS")

Commit message: Adjusted components according to availability in JLCPCB.
Parts:
- R11, R15, R35, R36, R37, R38, R39, R42, R43, R45, R46, R47, R48, R49, R50, R51, R52, R53: value 300R -> 330R
- R18, R19, R40, R41: value 2k2 -> 2,2k
- R21, R22, R23, R24, R25, R26, R27: value 2.2k -> 2,2k
- TP1: value 5VSH -> TP5019
- TP2: value 5V -> TP5019
- TP3: value GND -> TP5019
- TP8: value 3V3 -> TP5019
- moved FID2 170.2 mm to (136.0, 132.1)
- moved FID1 155.8 mm to (136.0, 70.1)
- moved FID4 89.5 mm to (215.5, 117.3)
- moved FID3 76.1 mm to (215.5, 70.1)

Commit message: Adjusted the footprint for the reset switch.
Parts:
- moved FID2 0.25 mm to (136.0, 132.3)
Routing:
- net GND: track 73.2 -> 71.8 mm, vias 77 -> 76
Changed lines of the file:
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@@
 	(footprint "Fiducial:Fiducial_1mm_Mask2mm"
 		(layer "F.Cu")
-		(at 136.02 132.08)
+		(at 136.02 132.33)
 		(descr "Fiducial, circular marking, 1mm bare copper, 2mm soldermask opening (Level A)")
 		(tags "fiducial")
@@
 		(sheetname "/MCU/")
 		(sheetfile "eumesmo-010-16ch-v1-mcu.kicad_sch")
-		(units
-			(unit
-				(name "A")
-				(pins "1" "2")
-			)
-		)
 		(attr smd)
 		(duplicate_pad_numbers_are_jumpers no)
 		(fp_line
 			(start 1.95 -1.5)
-			(end 1.95 1.5)
+			(end 1.95 -1.25)
 			(stroke
 				(width 0.12)
@@
 		)
 		(fp_line
+			(start -1.95 -1.25)
+			(end -1.95 -1.5)
+			(stroke
+				(width 0.12)
+				(type solid)
+			)
+			(layer "F.SilkS")
+		)
+		(fp_line
+			(start 1.95 1.5)
+			(end 1.95 1.25)
+			(stroke
+				(width 0.12)
+				(type solid)
+			)
+			(layer "F.SilkS")
+		)
+		(fp_line
 			(start 1.95 1.5)
 			(end -1.95 1.5)
@@
 		(fp_line
 			(start -1.95 1.5)
-			(end -1.95 -1.5)
+			(end -1.95 1.25)
 			(stroke
 				(width 0.12)
@@
 		)
 		(fp_line
-			(start 3.35 -1.6)
-			(end 3.35 1.6)
+			(start 2.85 -1.6)
+			(end 2.85 1.6)
 			(stroke
 				(width 0.05)
@@
 		)
 		(fp_line
-			(start -3.35 -1.6)
-			(end 3.35 -1.6)
+			(start -2.85 -1.6)
+			(end 2.85 -1.6)
 			(stroke
 				(width 0.05)
@@
 		)
 		(fp_line
-			(start 3.35 1.6)
-			(end -3.35 1.6)
+			(start 2.85 1.6)
+			(end -2.85 1.6)
 			(stroke
 				(width 0.05)
@@
 		)
 		(fp_line
-			(start -3.35 1.6)
-			(end -3.35 -1.6)
+			(start -2.85 1.6)
+			(end -2.85 -1.6)
 			(stroke
 				(width 0.05)
@@
 		)
 		(pad "1" smd rect
-			(at -2.75 0 90)
+			(at -2.225 0 90)
 			(size 1.05 2)
 			(layers "F.Cu" "F.Mask" "F.Paste")
@@
 		)
 		(pad "2" smd rect
-			(at 2.75 0 90)
+			(at 2.225 0 90)
 			(size 1.05 2)
 			(layers "F.Cu" "F.Mask" "F.Paste")
@@
 	)
 	(segment
-		(start 124.77 92.07)
-		(end 124.77 91.33)
-		(width 0.5)
+		(start 110.77 82.08)
+		(end 110.77 83.055)
+		(width 0.75)
 		(layer "F.Cu")
 		(net "GND")
 	)
 	(segment
-		(start 111.27 83.08)
-		(end 111.27 82.58)
+		(start 124.77 92.07)
+		(end 124.77 91.33)
 		(width 0.5)
 		(layer "F.Cu")
@@
 	)
 	(segment
-		(start 110.27 83.08)
-		(end 110.27 82.58)
-		(width 0.5)
-		(layer "F.Cu")
-		(net "GND")
-	)
-	(segment
 		(start 112.52 97.03)
 		(end 113.82 97.03)
@@
 	)
 	(segment
-		(start 110.77 83.58)
-		(end 110.27 83.08)
-		(width 0.5)
-		(layer "F.Cu")
-		(net "GND")
-	)
-	(segment
 		(start 117.77 94.33)
 		(end 117.77 95.13)
@@
 	)
 	(segment
-		(start 110.77 83.58)
-		(end 111.27 83.08)
-		(width 0.5)
-		(layer "F.Cu")
-		(net "GND")
-	)
-	(segment
 		(start 95.1325 78.08)
 		(end 94.27 78.08)
@@
 	)
 	(via
-		(at 110.27 82.58)
-		(size 0.6)
-		(drill 0.3)
-		(layers "F.Cu" "B.Cu")
-		(net "GND")
-	)
-	(via
 		(at 92.77 123.08)
 		(size 0.6)
@@
 	)
 	(via
-		(at 111.27 82.58)
+		(at 110.77 82.08)
 		(size 0.6)
 		(drill 0.3)
@@
 	)
 	(segment
+		(start 106.4075 79.08)
+		(end 108.77 79.08)
+		(width 0.3)
+		(layer "F.Cu")
+		(net "/MCU/UARTTXD")
+	)
+	(segment
 		(start 131.345 77.155)
 		(end 132.52 77.155)
@@
 		(net "/MCU/UARTTXD")
 	)
-	(segment
-		(start 106.4075 79.08)
-		(end 109.27 79.08)
-		(width 0.3)
-		(layer "F.Cu")
-		(net "/MCU/UARTTXD")
-	)
 	(via
 		(at 119.02 76.83)
@@
 	)
 	(via
-		(at 109.27 79.08)
+		(at 108.77 79.08)
 		(size 0.6)
 		(drill 0.3)
@@
 	)
 	(segment
-		(start 119.02 76.83)
+		(start 114.02 79.08)
 		(end 116.27 76.83)
 		(width 0.3)
@@
 	)
 	(segment
-		(start 116.27 76.83)
+		(start 108.77 79.08)
 		(end 114.02 79.08)
 		(width 0.3)
@@
 	)
 	(segment
-		(start 114.02 79.08)
-		(end 109.27 79.08)
+		(start 116.27 76.83)
+		(end 119.02 76.83)
 		(width 0.3)
 		(layer "B.Cu")
@@
 	)
 	(segment
-		(start 110.77 79.58)
-		(end 110.77 78.08)
+		(start 110.3825 76.9425)
+		(end 110.3825 76.53)
 		(width 0.5)
 		(layer "F.Cu")
@@
 	)
 	(segment
-		(start 108.77 76.34)
-		(end 109.53 76.34)
-		(width 0.5)
+		(start 107.42 82.93)
+		(end 104.6075 82.93)
+		(width 0.3)
 		(layer "F.Cu")
 		(net "/MCU/MRESET")
 	)
 	(segment
-		(start 110.3825 76.53)
-		(end 110.3825 76.9425)
+		(start 110.77 78.605)
+		(end 110.77 77.33)
 		(width 0.5)
 		(layer "F.Cu")
@@
 	)
 	(segment
-		(start 104.6075 82.93)
-		(end 107.42 82.93)
+		(start 110.77 78.605)
+		(end 110.77 79.58)
 		(width 0.3)
 		(layer "F.Cu")
@@
 	)
 	(segment
-		(start 110.77 77.33)
-		(end 110.77 78.08)
+		(start 108.77 76.34)
+		(end 109.53 76.34)
 		(width 0.5)
 		(layer "F.Cu")
@@
 	)
 	(segment
-		(start 107.42 82.93)
-		(end 110.77 79.58)
+		(start 110.77 79.58)
+		(end 107.42 82.93)
 		(width 0.3)
 		(layer "F.Cu")
@@
 	)
 	(segment
-		(start 110.3825 76.9425)
-		(end 110.77 77.33)
+		(start 110.77 77.33)
+		(end 110.3825 76.9425)
 		(width 0.5)
 		(layer "F.Cu")

Commit message: Text translated to english
Parts:
- U9: value TPS3823-33 -> TPS3820-33
