File: V1/eumesmo-010-16ch-analogs.kicad_sch (KiCad schematic)
At the start: 120 parts, among them U13 TLV274, U14 TLV274, U15 TLV274, U16 TLV274

Commit message: Development
Parts:
- added C69, C70, C71, C72, C73, C74, C75, C76, C77, C78, C79, C80, C81, C82, C83, C84: 100pF/50V, Tales:C_0805_2012Metric, symbol Device:C_Small
- R100, R109, R110, R119, R120, R129, R130, R59, R60, R69, R70, R79, R80, R89, R90, R99: value 10k/125mW -> 11k/125mW; LCSC Part # C17414 -> C17429; Mfr PN 0805W8F1002T5E -> 0805W8F1102T5E; Vendor PN C17414 -> C17429
- R104, R106, R114, R116, R124, R126, R54, R56, R64, R66, R74, R76, R84, R86, R94, R96: value 100k/125mW -> 10k/125mW; LCSC Part # C149504 -> C17414; Mfr PN 0805W8F1003T5E -> 0805W8F1002T5E; Vendor PN C149504 -> C17414
Connections:
- net CH01: no longer R59.2
- net CH01FB: now also C69.2
- net CH01OUT: now also R59.2, C69.1
- net CH02: no longer R60.2
- net CH02FB: now also C70.2
- net CH02OUT: now also R60.2, C70.1
- net CH03: no longer R69.2
- net CH03FB: now also C71.2
- net CH03OUT: now also R69.2, C71.1
- net CH04: no longer R70.2
- net CH04FB: now also C72.2
- net CH04OUT: now also R70.2, C72.1
- net CH05: no longer R79.2
- net CH05FB: now also C73.2
- net CH05OUT: now also R79.2, C73.1
- net CH06: no longer R80.2
- net CH06FB: now also C74.2
- net CH06OUT: now also R80.2, C74.1
- net CH07: no longer R89.2
- net CH07FB: now also C75.2
- net CH07OUT: now also R89.2, C75.1
- net CH08: no longer R90.2
- net CH08FB: now also C76.2
- net CH08OUT: now also R90.2, C76.1
- net CH09: no longer R99.2
- net CH09FB: now also C77.2
- net CH09OUT: now also R99.2, C77.1
- net CH10: no longer R100.2
- net CH10FB: now also C78.2
- net CH10OUT: now also R100.2, C78.1
- net CH11: no longer R109.2
- net CH11FB: now also C79.2
- net CH11OUT: now also R109.2, C79.1
- net CH12: no longer R110.2
- net CH12FB: now also C80.2
- net CH12OUT: now also R110.2, C80.1
- net CH13: no longer R119.2
- net CH13FB: now also C81.2
- net CH13OUT: now also R119.2, C81.1
- net CH14: no longer R120.2
- net CH14FB: now also C82.2
- net CH14OUT: now also R120.2, C82.1
- net CH15: no longer R129.2
- net CH15FB: now also C83.2
- net CH15OUT: now also R129.2, C83.1
- net CH16: no longer R130.2
- net CH16FB: now also C84.2
- net CH16OUT: now also R130.2, C84.1
Other:
- moved on the sheet: C33, C34, C37, C38, C41, C42, C49, C50, C53, C54, C57, C58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

Commit message: Development
Parts:
- renumbered C69 to C37, C70 to C38, C45 to C39, C46 to C40, C47 to C41, C48 to C42, C37 to C43, C38 to C44, C39 to C45, C40 to C46, C71 to C47, C72 to C48, C41 to C49, C42 to C50, C43 to C51, C44 to C52, C73 to C53, C74 to C54, C49 to C55, C50 to C56, C51 to C57, C52 to C58, C75 to C59, C76 to C60, C53 to C61, C54 to C62, C55 to C63, C56 to C64, C77 to C65, C78 to C66, C57 to C67, C58 to C68, C59 to C69, C60 to C70, C79 to C71, C80 to C72, C61 to C73, C62 to C74, C63 to C75, C64 to C76, C81 to C77, C82 to C78, C65 to C79, C66 to C80, C67 to C81, C68 to C82, R99 to R100, R100 to R101, R101 to R102, R102 to R103, R103 to R104, R104 to R105, R105 to R106, R106 to R107, R107 to R108, R108 to R109, R109 to R110, R110 to R111, R111 to R112, R112 to R113, R113 to R114, R114 to R115, R115 to R116, R116 to R117, R117 to R118, R118 to R119, R119 to R120, R120 to R121, R121 to R122, R122 to R123, R123 to R124, R124 to R125, R125 to R126, R126 to R127, R127 to R128, R128 to R129, R129 to R130, R130 to R131, R131 to R132, R132 to R133, R53 to R54, R54 to R55, R55 to R56, R56 to R57, R57 to R58, R58 to R59, R59 to R60, R60 to R61, R61 to R62, R62 to R63, R63 to R64, R64 to R65, R65 to R66, R66 to R67, R67 to R68, R68 to R69, R69 to R70, R70 to R71, R71 to R72, R72 to R73, R73 to R74, R74 to R75, R75 to R76, R76 to R77, R77 to R78, R78 to R79, R79 to R80, R80 to R81, R81 to R82, R82 to R83, R83 to R84, R84 to R85, R85 to R86, R86 to R87, R87 to R88, R88 to R89, R89 to R90, R90 to R91, R91 to R92, R92 to R93, R93 to R94, R94 to R95, R95 to R96, R96 to R97, R97 to R98, R98 to R99
Other:
- title: eumesmo 24V 16xIn/16xOut/1-Wire Module -> eumesmo 24V 16x 0-10V module
