File: V1/eumesmo-010-16ch-v1-lan.kicad_sch (KiCad schematic)
At the start: 29 parts, among them J8 ETHERNET, U6 LAN8710A, U7 TPS3823-33

Commit message: Development
Parts:
- U6: Technology (none) -> PHY
- U7: Technology (none) -> Voltage Monitor
Changed lines of the file:
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@@
 			)
 		)
+		(property "Technology" "Voltage Monitor"
+			(at 129.54 133.35 0)
+			(hide yes)
+			(show_name no)
+			(do_not_autoplace no)
+			(effects
+				(font
+					(size 1.27 1.27)
+				)
+			)
+		)
 		(pin "3"
 		)
@@
 			)
 		)
-		(property "Technology" ""
+		(property "Technology" "PHY"
 			(at 176.53 88.9 0)
 			(hide yes)

Commit message: Development
Parts:
- U9: renamed from U7; Case (none) -> SOT-23-5; JLCPCB BOM (none) -> 1; LCSC Part # (none) -> C7719; Mfr (none) -> Texas Instruments; Mfr PN (none) -> TPS3823-33DBVR; Vendor (none) -> JLCPCB; Vendor PN (none) -> C7719
- renumbered C19 to C22, C20 to C23, C21 to C24, C22 to C25, C23 to C26, C24 to C27, C25 to C28, J8 to J7, R21 to R19, R22 to R20, R23 to R21, R24 to R22, R25 to R23, R26 to R24, R27 to R25, R28 to R26, R29 to R27, R30 to R28, R31 to R29, R32 to R30, R33 to R31, R34 to R32, R35 to R33, U6 to U8

Commit message: Development
Parts:
- removed TP15: CLK, TestPoint:TestPoint_Pad_D1.5mm, symbol Connector:TestPoint
- renumbered D7 to D8, R19 to R20, R20 to R21, R21 to R22, R22 to R23, R23 to R24, R24 to R25, R25 to R26, R26 to R27, R27 to R28, R28 to R29, R29 to R30, R30 to R31, R31 to R32, R32 to R33, R33 to R34, TP14 to TP10, TP13 to TP9
Other:
- title: eumesmo 24V 16xIn/16xOut/1-Wire Module -> eumesmo 24V 16x 0-10V module
