File: V1/eumesmo-010-16ch-v1-lan.kicad_sch (KiCad schematic)
At the start: 28 parts, among them J7 ETHERNET, U8 LAN8710A, U9 TPS3820-33

Commit message: Component rotations and offsets ajusted for JLCPCB
Parts:
- D8: FT Rotation Offset (none) -> 90
- J7, U8: FT Rotation Offset (none) -> 180
Changed lines of the file:
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@@
+			)
+		)
+		(property "FT Rotation Offset" "180"
+			(at 48.26 154.94 0)
+			(hide yes)
+			(show_name no)
+			(do_not_autoplace no)
+			(effects
+				(font
+					(size 1.27 1.27)
+				)
 			)
 		)
@@
 			)
 		)
+		(property "FT Rotation Offset" "90"
+			(at 252.73 93.98 0)
+			(hide yes)
+			(show_name no)
+			(do_not_autoplace no)
+			(effects
+				(font
+					(size 1.27 1.27)
+				)
+			)
+		)
 		(pin "1"
 		)
@@
 			(at 176.53 88.9 0)
 			(hide yes)
+			(show_name no)
+			(do_not_autoplace no)
+			(effects
+				(font
+					(size 1.27 1.27)
+				)
+			)
+		)
+		(property "FT Rotation Offset" "180"
+			(at 176.53 88.9 0)
+			(hide yes)
