File: V1/eumesmo-010-16ch-v1.kicad_sch (KiCad schematic)
At the start: 8 parts, among them J1 250-208, J2 250-208, J3 250-208, J4 250-208

Commit message: Adjusted components according to availability in JLCPCB.
Parts:
- FID1, FID2, FID3, FID4: JLCPCB BOM 0 -> (none); now not fitted; now left out of the parts list
- J1, J2, J3, J4: JLCPCB BOM 1 -> (none)
Changed lines of the file:
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@@
 		(body_style 1)
 		(exclude_from_sim no)
-		(in_bom yes)
+		(in_bom no)
 		(on_board yes)
 		(in_pos_files yes)
-		(dnp no)
+		(dnp yes)
 		(fields_autoplaced yes)
 		(property "Reference" "FID1"
@@
 		)
 		(property "Description" "Fiducial Marker"
-			(at 22.86 171.45 0)
-			(hide yes)
-			(show_name no)
-			(do_not_autoplace no)
-			(effects
-				(font
-					(size 1.27 1.27)
-				)
-			)
-		)
-		(property "JLCPCB BOM" "0"
 			(at 22.86 171.45 0)
 			(hide yes)
@@
 		(body_style 1)
 		(exclude_from_sim no)
-		(in_bom yes)
+		(in_bom no)
 		(on_board yes)
 		(in_pos_files yes)
-		(dnp no)
+		(dnp yes)
 		(fields_autoplaced yes)
 		(property "Reference" "FID2"
@@
 		)
 		(property "Description" "Fiducial Marker"
-			(at 22.86 177.8 0)
-			(hide yes)
-			(show_name no)
-			(do_not_autoplace no)
-			(effects
-				(font
-					(size 1.27 1.27)
-				)
-			)
-		)
-		(property "JLCPCB BOM" "0"
 			(at 22.86 177.8 0)
 			(hide yes)
@@
 			)
 		)
-		(property "JLCPCB BOM" "1"
-			(at 219.71 144.78 0)
-			(hide yes)
-			(show_name no)
-			(do_not_autoplace no)
-			(effects
-				(font
-					(size 1.27 1.27)
-				)
-			)
-		)
 		(property "LCSC Part #" "C2833587"
 			(at 219.71 144.78 0)
@@
 			)
 		)
-		(property "JLCPCB BOM" "1"
-			(at 219.71 120.65 0)
-			(hide yes)
-			(show_name no)
-			(do_not_autoplace no)
-			(effects
-				(font
-					(size 1.27 1.27)
-				)
-			)
-		)
 		(property "LCSC Part #" "C2833587"
 			(at 219.71 120.65 0)
@@
 			)
 		)
-		(property "JLCPCB BOM" "1"
-			(at 219.71 95.25 0)
-			(hide yes)
-			(show_name no)
-			(do_not_autoplace no)
-			(effects
-				(font
-					(size 1.27 1.27)
-				)
-			)
-		)
 		(property "LCSC Part #" "C2833587"
 			(at 219.71 95.25 0)
@@
 		(body_style 1)
 		(exclude_from_sim no)
-		(in_bom yes)
+		(in_bom no)
 		(on_board yes)
 		(in_pos_files yes)
-		(dnp no)
+		(dnp yes)
 		(fields_autoplaced yes)
 		(property "Reference" "FID4"
@@
 		)
 		(property "Description" "Fiducial Marker"
-			(at 22.86 190.5 0)
-			(hide yes)
-			(show_name no)
-			(do_not_autoplace no)
-			(effects
-				(font
-					(size 1.27 1.27)
-				)
-			)
-		)
-		(property "JLCPCB BOM" "0"
 			(at 22.86 190.5 0)
 			(hide yes)
@@
 		(body_style 1)
 		(exclude_from_sim no)
-		(in_bom yes)
+		(in_bom no)
 		(on_board yes)
 		(in_pos_files yes)
-		(dnp no)
+		(dnp yes)
 		(fields_autoplaced yes)
 		(property "Reference" "FID3"
@@
 		)
 		(property "Description" "Fiducial Marker"
-			(at 22.86 184.15 0)
-			(hide yes)
-			(show_name no)
-			(do_not_autoplace no)
-			(effects
-				(font
-					(size 1.27 1.27)
-				)
-			)
-		)
-		(property "JLCPCB BOM" "0"
 			(at 22.86 184.15 0)
 			(hide yes)
@@
 			(at 219.71 71.12 0)
 			(hide yes)
-			(show_name no)
-			(do_not_autoplace no)
-			(effects
-				(font
-					(size 1.27 1.27)
-				)
-			)
-		)
-		(property "JLCPCB BOM" "1"
-			(at 219.71 71.12 0)
-			(hide yes)
